Commit message: full visual robot arm

File: robot_description/urdf/robot.xacro (robot description, xacro)
@@ -7,7 +7,11 @@
   <xacro:property name="LINK2" value="${params['link2_length']}"/>
   <xacro:property name="LINK3" value="${params['link3_length']}"/>
+  <xacro:property name="LINK4" value="${params['link4_length']}"/>
+  <xacro:property name="LINK5" value="${params['link5_length']}"/>
   <xacro:property name="LINK1_LENGTH" value="${LINK1-0.045}"/>
   <xacro:property name="LINK2_LENGTH" value="${LINK2-0.085}"/>
-  <xacro:property name="LINK3_LENGTH" value="${LINK3}"/>
+  <xacro:property name="LINK3_LENGTH" value="${LINK3-0.045-0.00625}"/>
+  <xacro:property name="LINK4_LENGTH" value="${LINK4-0.045}"/>
+  <xacro:property name="LINK5_LENGTH" value="${LINK5+0.015}"/>
   <material name="orange">
     <color rgba="${255/255} ${108/255} ${10/255} 1.0"/>
@@ -19,11 +23,11 @@
   <joint name="fixed" type="fixed">
     <parent link="world"/>
-    <child link="base_link"/>
-  </joint>
-  <link name="base_link">
-    <visual>
-      <origin xyz="0 0 0" rpy="0 0 0"/>
-      <geometry>
-        <mesh filename="file:///$(find robot_description)/meshes/link_base_m.STL"/>
+    <child link="link_slide"/>
+  </joint>
+  <link name="link_slide">
+    <visual>
+      <origin xyz="0 0 0" rpy="0 0 0"/>
+      <geometry>
+        <mesh filename="file:///$(find robot_description)/meshes/link_slide.STL"/>
       </geometry>
       <material name="white"/>
@@ -38,8 +42,32 @@
     </inertial>
   </link>
+  <joint name="joint0" type="prismatic">
+    <origin xyz="0.0 0.0 0.35" rpy="0.0 0.0 0.0"/>
+    <parent link="link_slide"/>
+    <child link="link0"/>
+    <axis xyz="1 0 0"/>
+    <limit lower="-0.75" upper="0.75" effort="0.0" velocity="0.0"/>
+  </joint>
+  <link name="link0">
+    <visual>
+      <origin xyz="0 0 0" rpy="0 0 0"/>
+      <geometry>
+        <mesh filename="file:///$(find robot_description)/meshes/link0.STL"/>
+      </geometry>
+      <material name="white"/>
+    </visual>
+    <inertial>
+      <origin xyz="0 0 0" rpy="0 0 0"/>
+      <mass value="0.5"/>
+      <inertia
+        ixx="0.0" ixy="0.0" ixz="0.0"
+        iyy="0.0" iyz="0.0"
+        izz="0.0"/>
+    </inertial>
+  </link>
   <joint name="joint1" type="revolute">
-    <parent link="base_link"/>
+    <parent link="link0"/>
     <child link="link1"/>
-    <origin rpy="0 0 0" xyz="0 0 0.04"/>
+    <origin rpy="0 0 0" xyz="0 0 0.2"/>
     <axis xyz="0 0 1"/>
     <limit lower="-3.14" upper="3.14" effort="1000" velocity="1000"/>
@@ -87,5 +115,5 @@
     <parent link="link_joint2-1"/>
     <child link="link_joint2-2" />
-    <origin rpy="${pi} ${pi/2} ${pi}" xyz="0.04 0 ${LINK1_LENGTH+0.045}"/>
+    <origin rpy="${pi} ${pi/2} 0" xyz="0.04 0 ${LINK1_LENGTH+0.045}"/>
     <axis xyz="0 0 1"/>
     <limit lower="-3.14" upper="3.14" effort="1000" velocity="1000"/>
@@ -94,5 +122,5 @@
   <link name="link_joint2-2">
     <visual>
-      <origin xyz="0 0 0.04" rpy="${pi} 0 ${pi}"/>
+      <origin xyz="0 0 -0.04" rpy="0 0 ${pi}"/>
       <geometry>
         <mesh filename="file:///$(find robot_description)/meshes/joint_2-2.STL"/>
@@ -112,5 +140,5 @@
     <parent link="link_joint2-2"/>
     <child link="link2"/>
-    <origin rpy="0 ${-pi/2} 0" xyz="${(-LINK2_LENGTH/2)-0.005} 0 0.04"/>
+    <origin rpy="0 ${-pi/2} ${-pi}" xyz="${(-LINK2_LENGTH/2)-0.085} 0 -0.04"/>
   </joint>
   <link name="link2">
@@ -134,5 +162,5 @@
     <parent link="link2"/>
     <child link="link_joint3-1"/>
-    <origin rpy="0 ${-pi/2} 0" xyz="0 0 ${(LINK2_LENGTH/2)+0.085}"/>
+    <origin rpy="0 ${pi/2} 0" xyz="0 0 ${-(LINK2_LENGTH/2)-0.005}"/>
   </joint>
   <link name="link_joint3-1">
@@ -232,7 +260,7 @@
   <link name="link4">
     <visual>
-      <origin xyz="0 0 0.0725" rpy="0 0 0"/>
-      <geometry>
-        <cylinder radius="0.035" length="0.145"/>
+      <origin xyz="0 0 ${LINK4_LENGTH/2}" rpy="0 0 0"/>
+      <geometry>
+        <cylinder radius="0.035" length="${LINK4_LENGTH}"/>
       </geometry>
       <material name="white"/>
@@ -250,5 +278,5 @@
     <parent link="link4"/>
     <child link="link_joint5"/>
-    <origin rpy="0 ${-pi/2} 0" xyz="0 0 0.19"/>
+    <origin rpy="0 ${-pi/2} 0" xyz="0 0 ${LINK4_LENGTH+0.045}"/>
   </joint>
   <link name="link_joint5">
@@ -260,7 +288,15 @@
       <material name="orange"/>
     </visual>
-  </link>
-  <!-- <joint name="joint5" type="revolute">
-    <parent link="link_joint4"/>
+    <inertial>
+      <origin xyz="0 0 0" rpy="0 0 0"/>
+      <mass value="0.1"/>
+      <inertia
+        ixx="0.0" ixy="0.0" ixz="0.0"
+        iyy="0.0" iyz="0.0"
+        izz="0.0"/>
+    </inertial>
+  </link>
+  <joint name="joint5" type="revolute">
+    <parent link="link_joint5"/>
     <child link="link5" />
     <origin rpy="0 0 0" xyz="0 0 0"/>
@@ -271,7 +307,7 @@
   <link name="link5">
     <visual>
-      <origin xyz="0.5 0 0" rpy="0 0 0"/>
-      <geometry>
-        <cylinder radius="0.03" length="0.118"/>
+      <origin xyz="${(LINK5_LENGTH/2)-0.015} 0 0" rpy="0 ${pi/2} 0"/>
+      <geometry>
+        <cylinder radius="0.03" length="${LINK5_LENGTH}"/>
       </geometry>
       <material name="white"/>
@@ -286,8 +322,8 @@
     </inertial>
   </link>
-  <joint name="joint6" type="fixed">
+  <joint name="joint6" type="revolute">
     <parent link="link5"/>
     <child link="hook" />
-    <origin rpy="0 ${pi/2} 0" xyz="0.0905 0 0"/>
+    <origin rpy="0 ${pi/2} 0" xyz="${(LINK5_LENGTH)-0.015+0.0265} 0 0"/>
     <axis xyz="0 0 1"/>
     <limit lower="-3.14" upper="3.14" effort="1000" velocity="1000"/>
@@ -302,5 +338,13 @@
       <material name="orange"/>
     </visual>
-  </link> -->
+    <inertial>
+      <origin xyz="0 0 0" rpy="0 0 0"/>
+      <mass value="0.1"/>
+      <inertia
+        ixx="0.0" ixy="0.0" ixz="0.0"
+        iyy="0.0" iyz="0.0"
+        izz="0.0"/>
+    </inertial>
+  </link>
   <!-- <xacro:include filename="gazebo.xacro" /> -->
   <!-- gazebo plugin -->
@@ -309,10 +353,11 @@
           filename="libgazebo_ros_joint_state_publisher.so">
           <update_rate>20</update_rate>
+          <joint_name>joint0</joint_name>
           <joint_name>joint1</joint_name>
           <joint_name>joint2</joint_name>
           <joint_name>joint3</joint_name>
           <joint_name>joint4</joint_name>
-          <!-- <joint_name>joint5</joint_name>
-          <joint_name>joint6</joint_name> -->
+          <joint_name>joint5</joint_name>
+          <joint_name>joint6</joint_name>
       </plugin>
   </gazebo>
@@ -321,5 +366,52 @@
       <plugin>gazebo_ros2_control/GazeboSystem</plugin>
     </hardware>
+    <joint name="joint0">
+        <command_interface name="position">
+          <param name="min">-0.75</param>
+          <param name="max">0.75</param>
+        </command_interface>
+        <state_interface name="position">
+            <param name="initial_value">0.0</param>
+        </state_interface>
+    </joint>
     <joint name="joint1">
+        <command_interface name="position">
+          <param name="min">-3.14</param>
+          <param name="max">3.14</param>
+        </command_interface>
+        <state_interface name="position">
+            <param name="initial_value">0.0</param>
+        </state_interface>
+        <!-- <state_interface name="velocity"/>
+        <state_interface name="effort"/> -->
+    </joint>
+    <joint name="joint2">
+        <command_interface name="position">
+          <param name="min">-3.14</param>
+          <param name="max">3.14</param>
+        </command_interface>
+        <state_interface name="position">
+            <param name="initial_value">0.0</param>
+        </state_interface>
+    </joint>
+    <joint name="joint3">
+        <command_interface name="position">
+          <param name="min">-3.14</param>
+          <param name="max">3.14</param>
+        </command_interface>
+        <state_interface name="position">
+            <param name="initial_value">0.0</param>
+        </state_interface>
+    </joint>
+    <joint name="joint4">
+        <command_interface name="position">
+          <param name="min">-3.14</param>
+          <param name="max">3.14</param>
+        </command_interface>
+        <state_interface name="position">
+            <param name="initial_value">0.0</param>
+        </state_interface>
+    </joint>
+    <joint name="joint5">
         <command_interface name="position">
           <param name="min">-1</param>
@@ -329,52 +421,14 @@
             <param name="initial_value">0.0</param>
         </state_interface>
-        <!-- <state_interface name="velocity"/>
-        <state_interface name="effort"/> -->
-    </joint>
-    <joint name="joint2">
-        <command_interface name="position">
-          <param name="min">-1</param>
-          <param name="max">1</param>
-        </command_interface>
-        <state_interface name="position">
-            <param name="initial_value">0.0</param>
-        </state_interface>
-    </joint>
-    <joint name="joint3">
-        <command_interface name="position">
-          <param name="min">-1</param>
-          <param name="max">1</param>
-        </command_interface>
-        <state_interface name="position">
-            <param name="initial_value">0.0</param>
-        </state_interface>
-    </joint>
-    <joint name="joint4">
-        <command_interface name="position">
-          <param name="min">-1</param>
-          <param name="max">1</param>
-        </command_interface>
-        <state_interface name="position">
-            <param name="initial_value">0.0</param>
-        </state_interface>
-    </joint>
-    <!-- <joint name="joint5">
-        <command_interface name="position">
-          <param name="min">-1</param>
-          <param name="max">1</param>
-        </command_interface>
-        <state_interface name="position">
-            <param name="initial_value">0.0</param>
-        </state_interface>
     </joint>
     <joint name="joint6">
         <command_interface name="position">
-          <param name="min">-1</param>
-          <param name="max">1</param>
-        </command_interface>
-        <state_interface name="position">
-            <param name="initial_value">0.0</param>
-        </state_interface>
-    </joint> -->
+          <param name="min">-3.14</param>
+          <param name="max">3.14</param>
+        </command_interface>
+        <state_interface name="position">
+            <param name="initial_value">0.0</param>
+        </state_interface>
+    </joint>
   </ros2_control>
   <gazebo>
@@ -384,8 +438,10 @@
   </gazebo>
   <!-- Base Link -->
-  <gazebo reference="base_link">
-    <material>Gazebo/White</material>
-  </gazebo>
-  <!-- Link1 -->
+  <gazebo reference="link_slide">
+    <material>Gazebo/White</material>
+  </gazebo>
+  <gazebo reference="link0">
+    <material>Gazebo/White</material>
+  </gazebo>
   <gazebo reference="link1">
     <material>Gazebo/White</material>
@@ -418,9 +474,9 @@
     <material>Gazebo/Orange</material>
   </gazebo>
-  <!-- <gazebo reference="link5">
+  <gazebo reference="link5">
     <material>Gazebo/White</material>
   </gazebo>
   <gazebo reference="hook">
     <material>Gazebo/Orange</material>
-  </gazebo> -->
+  </gazebo>
 </robot>

Commit message: add environment

File: robot_description/urdf/robot.xacro (robot description, xacro)
@@ -20,6 +20,58 @@
     <color rgba="1.0 1.0 1.0 1.0"/>
   </material>
+  <material name="blue">
+    <color rgba="${118/255} ${186/255} ${255/255} 0.62"/>
+  </material>
   <link name="world"/>
-  <joint name="fixed" type="fixed">
+  <joint name="fixed_shelf" type="fixed">
+    <parent link="world"/>
+    <child link="shelf"/>
+  </joint>
+  <link name="shelf">
+    <visual>
+      <origin xyz="0 0.1 0" rpy="0 0 0"/>
+      <geometry>
+        <mesh filename="file:///$(find robot_description)/meshes/shelf.STL"/>
+      </geometry>
+      <material name="white"/>
+    </visual>
+    <inertial>
+      <origin xyz="0 0.1 0" rpy="0 0 0"/>
+      <mass value="5.0"/>
+      <inertia
+        ixx="0.01" ixy="0.0" ixz="0.0"
+        iyy="0.01" iyz="0.0"
+        izz="0.01"/>
+    </inertial>
+    <collision>
+      <origin xyz="0 0.1 0" rpy="0 0 0"/>
+      <geometry>
+        <mesh filename="file:///$(find robot_description)/meshes/shelf.STL"/>
+      </geometry>
+    </collision>
+  </link>
+  <joint name="float_obj1" type="floating">
+    <parent link="shelf"/>
+    <child link="obj1"/>
+  </joint>
+  <link name="obj1">
+    <visual>
+      <origin xyz="-0.44 0.32 0.4" rpy="0 0 0"/>
+      <geometry>
+        <cylinder radius="0.04" length="0.1"/>
+      </geometry>
+      <material name="blue"/>
+    </visual>
+    <inertial>
+      <origin xyz="-0.44 0.32 0.4" rpy="0 0 0"/>
+      <mass value="0.01"/>
+      <inertia
+        ixx="0.01" ixy="0.0" ixz="0.0"
+        iyy="0.01" iyz="0.0"
+        izz="0.01"/>
+    </inertial>
+  </link>
+  <!-- robot -->
+  <joint name="fixed_robot" type="fixed">
     <parent link="world"/>
     <child link="link_slide"/>
@@ -37,15 +89,22 @@
       <mass value="0.5"/>
       <inertia
-        ixx="0.0" ixy="0.0" ixz="0.0"
-        iyy="0.0" iyz="0.0"
-        izz="0.0"/>
-    </inertial>
+        ixx="0.01" ixy="0.0" ixz="0.0"
+        iyy="0.01" iyz="0.0"
+        izz="0.01"/>
+    </inertial>
+    <collision>
+      <origin xyz="0 0 0" rpy="0 0 0"/>
+      <geometry>
+        <!-- <box size="1.0 0.2 0.2"/> -->
+        <mesh filename="file:///$(find robot_description)/meshes/link_slide.STL"/>
+      </geometry>
+    </collision>
   </link>
   <joint name="joint0" type="prismatic">
-    <origin xyz="0.0 0.0 0.35" rpy="0.0 0.0 0.0"/>
+    <origin xyz="0.0 0.0 0.2" rpy="0.0 0.0 0.0"/>
     <parent link="link_slide"/>
     <child link="link0"/>
     <axis xyz="1 0 0"/>
-    <limit lower="-0.75" upper="0.75" effort="0.0" velocity="0.0"/>
+    <limit lower="-0.40" upper="0.40" effort="0.0" velocity="0.0"/>
   </joint>
   <link name="link0">
@@ -53,5 +112,5 @@
       <origin xyz="0 0 0" rpy="0 0 0"/>
       <geometry>
-        <mesh filename="file:///$(find robot_description)/meshes/link0.STL"/>
+        <mesh filename="file:///$(find robot_description)/meshes/link_base.STL"/>
       </geometry>
       <material name="white"/>
@@ -61,13 +120,19 @@
       <mass value="0.5"/>
       <inertia
-        ixx="0.0" ixy="0.0" ixz="0.0"
-        iyy="0.0" iyz="0.0"
-        izz="0.0"/>
-    </inertial>
+        ixx="0.01" ixy="0.0" ixz="0.0"
+        iyy="0.01" iyz="0.0"
+        izz="0.01"/>
+    </inertial>
+    <!-- <collision>
+      <origin xyz="0.0 0.0 0.0" rpy="0.0 0.0 0.0"/>
+      <geometry>
+        <mesh filename="file:///$(find robot_description)/meshes/link_base.STL"/>
+      </geometry>
+    </collision> -->
   </link>
   <joint name="joint1" type="revolute">
     <parent link="link0"/>
     <child link="link1"/>
-    <origin rpy="0 0 0" xyz="0 0 0.2"/>
+    <origin rpy="0 0 0" xyz="0 0 0.04"/>
     <axis xyz="0 0 1"/>
     <limit lower="-3.14" upper="3.14" effort="1000" velocity="1000"/>
@@ -86,7 +151,7 @@
       <mass value="0.5"/>
       <inertia
-        ixx="0.0" ixy="0.0" ixz="0.0"
-        iyy="0.0" iyz="0.0"
-        izz="0.0"/>
+        ixx="0.01" ixy="0.0" ixz="0.0"
+        iyy="0.01" iyz="0.0"
+        izz="0.01"/>
     </inertial>
   </link>
@@ -107,7 +172,7 @@
       <mass value="0.5"/>
       <inertia
-        ixx="0.0" ixy="0.0" ixz="0.0"
-        iyy="0.0" iyz="0.0"
-        izz="0.0"/>
+        ixx="0.01" ixy="0.0" ixz="0.0"
+        iyy="0.01" iyz="0.0"
+        izz="0.01"/>
     </inertial>
   </link>
@@ -132,7 +197,7 @@
       <mass value="0.01"/>
       <inertia
-        ixx="0.0" ixy="0.0" ixz="0.0"
-        iyy="0.0" iyz="0.0"
-        izz="0.0"/>
+        ixx="0.01" ixy="0.0" ixz="0.0"
+        iyy="0.01" iyz="0.0"
+        izz="0.01"/>
     </inertial>
   </link>
@@ -154,7 +219,7 @@
       <mass value="0.0"/>
       <inertia
-        ixx="0.0" ixy="0.0" ixz="0.0"
-        iyy="0.0" iyz="0.0"
-        izz="0.0"/>
+        ixx="0.01" ixy="0.0" ixz="0.0"
+        iyy="0.01" iyz="0.0"
+        izz="0.01"/>
     </inertial>
   </link>
@@ -176,7 +241,7 @@
       <mass value="0.1"/>
       <inertia
-        ixx="0.0" ixy="0.0" ixz="0.0"
-        iyy="0.0" iyz="0.0"
-        izz="0.0"/>
+        ixx="0.01" ixy="0.0" ixz="0.0"
+        iyy="0.01" iyz="0.0"
+        izz="0.01"/>
     </inertial>
   </link>
@@ -201,7 +266,7 @@
       <mass value="0.01"/>
       <inertia
-        ixx="0.0" ixy="0.0" ixz="0.0"
-        iyy="0.0" iyz="0.0"
-        izz="0.0"/>
+        ixx="0.01" ixy="0.0" ixz="0.0"
+        iyy="0.01" iyz="0.0"
+        izz="0.01"/>
     </inertial>
   </link>
@@ -223,7 +288,7 @@
       <mass value="0.01"/>
       <inertia
-        ixx="0.0" ixy="0.0" ixz="0.0"
-        iyy="0.0" iyz="0.0"
-        izz="0.0"/>
+        ixx="0.01" ixy="0.0" ixz="0.0"
+        iyy="0.01" iyz="0.0"
+        izz="0.01"/>
     </inertial>
   </link>
@@ -245,7 +310,7 @@
       <mass value="0.1"/>
       <inertia
-        ixx="0.0" ixy="0.0" ixz="0.0"
-        iyy="0.0" iyz="0.0"
-        izz="0.0"/>
+        ixx="0.01" ixy="0.0" ixz="0.0"
+        iyy="0.01" iyz="0.0"
+        izz="0.01"/>
     </inertial>
   </link>
@@ -270,7 +335,7 @@
       <mass value="0.01"/>
       <inertia
-        ixx="0.0" ixy="0.0" ixz="0.0"
-        iyy="0.0" iyz="0.0"
-        izz="0.0"/>
+        ixx="0.01" ixy="0.0" ixz="0.0"
+        iyy="0.01" iyz="0.0"
+        izz="0.01"/>
     </inertial>
   </link>
@@ -292,7 +357,7 @@
       <mass value="0.1"/>
       <inertia
-        ixx="0.0" ixy="0.0" ixz="0.0"
-        iyy="0.0" iyz="0.0"
-        izz="0.0"/>
+        ixx="0.01" ixy="0.0" ixz="0.0"
+        iyy="0.01" iyz="0.0"
+        izz="0.01"/>
     </inertial>
   </link>
@@ -317,12 +382,12 @@
       <mass value="0.01"/>
       <inertia
-        ixx="0.0" ixy="0.0" ixz="0.0"
-        iyy="0.0" iyz="0.0"
-        izz="0.0"/>
+        ixx="0.01" ixy="0.0" ixz="0.0"
+        iyy="0.01" iyz="0.0"
+        izz="0.01"/>
     </inertial>
   </link>
   <joint name="joint6" type="revolute">
     <parent link="link5"/>
-    <child link="hook" />
+    <child link="link_hook" />
     <origin rpy="0 ${pi/2} 0" xyz="${(LINK5_LENGTH)-0.015+0.0265} 0 0"/>
     <axis xyz="0 0 1"/>
@@ -330,9 +395,9 @@
     <dynamics damping="0" friction="1"/>
   </joint>
-  <link name="hook">
-    <visual>
-      <origin xyz="0 0 0" rpy="0 0 0"/>
-      <geometry>
-        <mesh filename="file:///$(find robot_description)/meshes/hook.STL"/>
+  <link name="link_hook">
+    <visual>
+      <origin xyz="0 0 0" rpy="0 0 0"/>
+      <geometry>
+        <mesh filename="file:///$(find robot_description)/meshes/link_hook.STL"/>
       </geometry>
       <material name="orange"/>
@@ -342,8 +407,71 @@
       <mass value="0.1"/>
       <inertia
-        ixx="0.0" ixy="0.0" ixz="0.0"
-        iyy="0.0" iyz="0.0"
-        izz="0.0"/>
-    </inertial>
+        ixx="0.01" ixy="0.0" ixz="0.0"
+        iyy="0.01" iyz="0.0"
+        izz="0.01"/>
+    </inertial>
+  </link>
+  <joint name="fixed_collision_box1" type="fixed">
+    <parent link="link_hook"/>
+    <child link="collision_box_1"/>
+    <origin rpy="0 0 0" xyz="0 0 0"/>
+  </joint>
+  <link name="collision_box_1">
+    <inertial>
+      <origin xyz="0 0 -0.0125" rpy="0 0 0"/>
+      <mass value="0.01"/>
+      <inertia
+        ixx="0.01" ixy="0.0" ixz="0.0"
+        iyy="0.01" iyz="0.0"
+        izz="0.01"/>
+    </inertial>
+    <collision>
+      <origin xyz="0 0 -0.0125" rpy="0 0 0"/>
+      <geometry>
+        <box size="0.08 0.08 0.025"/>
+      </geometry>
+    </collision>
+  </link>
+  <joint name="fixed_collision_box2" type="fixed">
+    <parent link="collision_box_1"/>
+    <child link="collision_box_2"/>
+    <origin rpy="0 0 0" xyz="0 0 0"/>
+  </joint>
+  <link name="collision_box_2">
+    <inertial>
+      <origin xyz="-0.05 0 0.035" rpy="0 0 0"/>
+      <mass value="0.01"/>
+      <inertia
+        ixx="0.01" ixy="0.0" ixz="0.0"
+        iyy="0.01" iyz="0.0"
+        izz="0.01"/>
+    </inertial>
+    <collision>
+      <origin xyz="-0.05 0 0.035" rpy="0 0 0"/>
+      <geometry>
+        <box size="0.02 0.08 0.11"/>
+      </geometry>
+    </collision>
+  </link>
+  <joint name="fixed_collision_box3" type="fixed">
+    <parent link="collision_box_2"/>
+    <child link="collision_box_3"/>
+    <origin rpy="0 0 0" xyz="0 0 0"/>
+  </joint>
+  <link name="collision_box_3">
+    <inertial>
+      <origin xyz="-0.01 0 0.1" rpy="0 0 0"/>
+      <mass value="0.01"/>
+      <inertia
+        ixx="0.01" ixy="0.0" ixz="0.0"
+        iyy="0.01" iyz="0.0"
+        izz="0.01"/>
+    </inertial>
+    <collision>
+      <origin xyz="-0.01 0 0.1" rpy="0 0 0"/>
+      <geometry>
+        <box size="0.1 0.08 0.02"/>
+      </geometry>
+    </collision>
   </link>
   <!-- <xacro:include filename="gazebo.xacro" /> -->
@@ -383,6 +511,4 @@
             <param name="initial_value">0.0</param>
         </state_interface>
-        <!-- <state_interface name="velocity"/>
-        <state_interface name="effort"/> -->
     </joint>
     <joint name="joint2">
@@ -433,9 +559,15 @@
   </ros2_control>
   <gazebo>
-    <plugin name="gazebo_ros_control" filename="libgazebo_ros_control.so">
+    <plugin name="gazebo_ros2_control" filename="libgazebo_ros2_control.so">
       <parameters>$(find robot_description)/config/controller.yaml</parameters>
     </plugin>
   </gazebo>
   <!-- Base Link -->
+  <gazebo reference="shelf">
+    <material>Gazebo/White</material>
+  </gazebo>
+  <gazebo reference="obj1">
+    <material>Gazebo/Blue</material>
+  </gazebo>
   <gazebo reference="link_slide">
     <material>Gazebo/White</material>
@@ -477,5 +609,5 @@
     <material>Gazebo/White</material>
   </gazebo>
-  <gazebo reference="hook">
+  <gazebo reference="link_hook">
     <material>Gazebo/Orange</material>
   </gazebo>
