Commit message: length limit

File: robot_description/urdf/robot.xacro (robot description, xacro)
@@ -9,4 +9,34 @@
   <xacro:property name="LINK4" value="${params['link4_length']}"/>
   <xacro:property name="LINK5" value="${params['link5_length']}"/>
+  <xacro:if value="${LINK1 >= 0.5}">
+    <xacro:property name="LINK1" value="0.5"/>
+  </xacro:if>
+  <xacro:if value="${0.045 >= LINK1}">
+    <xacro:property name="LINK1" value="0.045"/>
+  </xacro:if>
+  <xacro:if value="${LINK2 >= 0.5}">
+    <xacro:property name="LINK2" value="0.5"/>
+  </xacro:if>
+  <xacro:if value="${0.085 >= LINK2}">
+    <xacro:property name="LINK2" value="0.085"/>
+  </xacro:if>
+  <xacro:if value="${LINK3 >= 0.5}">
+    <xacro:property name="LINK3" value="0.5"/>
+  </xacro:if>
+  <xacro:if value="${0.05125 >= LINK3}">
+    <xacro:property name="LINK3" value="0.05125"/>
+  </xacro:if>
+  <xacro:if value="${LINK4 >= 0.5}">
+    <xacro:property name="LINK4" value="0.5"/>
+  </xacro:if>
+  <xacro:if value="${0.045 >= LINK4}">
+    <xacro:property name="LINK4" value="0.045"/>
+  </xacro:if>
+  <xacro:if value="${LINK5 >= 0.5}">
+    <xacro:property name="LINK5" value="0.5"/>
+  </xacro:if>
+  <xacro:if value="${0.0115 >= LINK5}">
+    <xacro:property name="LINK5" value="0.0115"/>
+  </xacro:if>
   <xacro:property name="LINK1_LENGTH" value="${LINK1-0.045}"/>
   <xacro:property name="LINK2_LENGTH" value="${LINK2-0.085}"/>
@@ -54,8 +84,10 @@
     <parent link="shelf"/>
     <child link="obj1"/>
+    <dynamics damping="0.0" friction="10.0"/>
+    <limit effort="1" velocity="1.0" lower="-2.2" upper="0.7" />
   </joint>
   <link name="obj1">
     <visual>
-      <origin xyz="-0.44 0.32 0.4" rpy="0 0 0"/>
+      <origin xyz="-0.6 0.35 0.45" rpy="0 0 0"/>
       <geometry>
         <cylinder radius="0.04" length="0.1"/>
@@ -64,11 +96,71 @@
     </visual>
     <inertial>
-      <origin xyz="-0.44 0.32 0.4" rpy="0 0 0"/>
-      <mass value="0.01"/>
-      <inertia
-        ixx="0.01" ixy="0.0" ixz="0.0"
-        iyy="0.01" iyz="0.0"
-        izz="0.01"/>
-    </inertial>
+      <origin xyz="-0.6 0.35 0.45" rpy="0 0 0"/>
+      <mass value="0.01"/>
+      <inertia
+        ixx="0.01" ixy="0.0" ixz="0.0"
+        iyy="0.01" iyz="0.0"
+        izz="0.01"/>
+    </inertial>
+    <collision>
+      <origin xyz="-0.6 0.35 0.45" rpy="0 0 0"/>
+      <geometry>
+        <cylinder radius="0.04" length="0.1"/>
+      </geometry>
+    </collision>
+  </link>
+  <joint name="float_obj2" type="floating">
+    <parent link="shelf"/>
+    <child link="obj2"/>
+  </joint>
+  <link name="obj2">
+    <visual>
+      <origin xyz="-0.3 0.35 0.45" rpy="0 0 0"/>
+      <geometry>
+        <cylinder radius="0.04" length="0.1"/>
+      </geometry>
+      <material name="blue"/>
+    </visual>
+    <inertial>
+      <origin xyz="-0.3 0.35 0.45" rpy="0 0 0"/>
+      <mass value="0.01"/>
+      <inertia
+        ixx="0.01" ixy="0.0" ixz="0.0"
+        iyy="0.01" iyz="0.0"
+        izz="0.01"/>
+    </inertial>
+    <collision>
+      <origin xyz="-0.3 0.35 0.45" rpy="0 0 0"/>
+      <geometry>
+        <cylinder radius="0.04" length="0.1"/>
+      </geometry>
+    </collision>
+  </link>
+  <joint name="float_obj8" type="floating">
+    <parent link="shelf"/>
+    <child link="obj8"/>
+  </joint>
+  <link name="obj8">
+    <visual>
+      <origin xyz="0.0 0.35 0.85" rpy="0 0 0"/>
+      <geometry>
+        <cylinder radius="0.04" length="0.1"/>
+      </geometry>
+      <material name="blue"/>
+    </visual>
+    <inertial>
+      <origin xyz="0.0 0.35 0.85" rpy="0 0 0"/>
+      <mass value="0.01"/>
+      <inertia
+        ixx="0.01" ixy="0.0" ixz="0.0"
+        iyy="0.01" iyz="0.0"
+        izz="0.01"/>
+    </inertial>
+    <collision>
+      <origin xyz="0.0 0.35 0.85" rpy="0 0 0"/>
+      <geometry>
+        <cylinder radius="0.04" length="0.1"/>
+      </geometry>
+    </collision>
   </link>
   <!-- robot -->
@@ -183,5 +275,5 @@
     <axis xyz="0 0 1"/>
     <limit lower="-3.14" upper="3.14" effort="1000" velocity="1000"/>
-    <dynamics damping="0" friction="1"/>
+    <dynamics damping="0" friction="1000"/>
   </joint>
   <link name="link_joint2-2">
@@ -252,5 +344,5 @@
     <axis xyz="0 0 1"/>
     <limit lower="-3.14" upper="3.14" effort="1000" velocity="1000"/>
-    <dynamics damping="0" friction="1"/>
+    <dynamics damping="0" friction="1000"/>
   </joint>
   <link name="link_joint3-2">
@@ -321,5 +413,5 @@
     <axis xyz="0 0 1"/>
     <limit lower="-3.14" upper="3.14" effort="1000" velocity="1000"/>
-    <dynamics damping="0" friction="1"/>
+    <dynamics damping="0" friction="1000"/>
   </joint>
   <link name="link4">
@@ -368,5 +460,5 @@
     <axis xyz="0 0 1"/>
     <limit lower="-1" upper="1" effort="1000" velocity="1000"/>
-    <dynamics damping="0" friction="1"/>
+    <dynamics damping="0" friction="1000"/>
   </joint>
   <link name="link5">
@@ -393,5 +485,5 @@
     <axis xyz="0 0 1"/>
     <limit lower="-3.14" upper="3.14" effort="1000" velocity="1000"/>
-    <dynamics damping="0" friction="1"/>
+    <dynamics damping="0" friction="1000"/>
   </joint>
   <link name="link_hook">
@@ -570,4 +662,10 @@
     <material>Gazebo/Blue</material>
   </gazebo>
+  <gazebo reference="obj2 ">
+    <material>Gazebo/Blue</material>
+  </gazebo>
+  <gazebo reference="obj8">
+    <material>Gazebo/Blue</material>
+  </gazebo>
   <gazebo reference="link_slide">
     <material>Gazebo/White</material>

Commit message: add parameter

File: robot_description/urdf/robot.xacro (robot description, xacro)
@@ -2,4 +2,5 @@
 <robot name="robot" xmlns:xacro="http://www.ros.org/wiki/xacro">
   <xacro:property name="PI" value="3.1415926535897931"/>
+  <xacro:property name="shelf_dist" value="0.1"/>
   <xacro:property name="params_path" value="$(find robot_description)/config/properties.yaml"/>
   <xacro:property name="params" value="${xacro.load_yaml(params_path)}"/>
@@ -9,33 +10,43 @@
   <xacro:property name="LINK4" value="${params['link4_length']}"/>
   <xacro:property name="LINK5" value="${params['link5_length']}"/>
-  <xacro:if value="${LINK1 >= 0.5}">
-    <xacro:property name="LINK1" value="0.5"/>
-  </xacro:if>
-  <xacro:if value="${0.045 >= LINK1}">
-    <xacro:property name="LINK1" value="0.045"/>
-  </xacro:if>
-  <xacro:if value="${LINK2 >= 0.5}">
-    <xacro:property name="LINK2" value="0.5"/>
-  </xacro:if>
-  <xacro:if value="${0.085 >= LINK2}">
-    <xacro:property name="LINK2" value="0.085"/>
-  </xacro:if>
-  <xacro:if value="${LINK3 >= 0.5}">
-    <xacro:property name="LINK3" value="0.5"/>
-  </xacro:if>
-  <xacro:if value="${0.05125 >= LINK3}">
-    <xacro:property name="LINK3" value="0.05125"/>
-  </xacro:if>
-  <xacro:if value="${LINK4 >= 0.5}">
-    <xacro:property name="LINK4" value="0.5"/>
-  </xacro:if>
-  <xacro:if value="${0.045 >= LINK4}">
-    <xacro:property name="LINK4" value="0.045"/>
-  </xacro:if>
-  <xacro:if value="${LINK5 >= 0.5}">
-    <xacro:property name="LINK5" value="0.5"/>
-  </xacro:if>
-  <xacro:if value="${0.0115 >= LINK5}">
-    <xacro:property name="LINK5" value="0.0115"/>
+  <xacro:property name="MAX_LINK1" value="0.2"/>
+  <xacro:property name="MAX_LINK2" value="0.2"/>
+  <xacro:property name="MAX_LINK3" value="0.2"/>
+  <xacro:property name="MAX_LINK4" value="0.2"/>
+  <xacro:property name="MAX_LINK5" value="0.2"/>
+  <xacro:property name="MIN_LINK1" value="0.045"/>
+  <xacro:property name="MIN_LINK2" value="0.085"/>
+  <xacro:property name="MIN_LINK3" value="0.05125"/>
+  <xacro:property name="MIN_LINK4" value="0.045"/>
+  <xacro:property name="MIN_LINK5" value="0.0115"/>
+  <xacro:if value="${LINK1 >= MAX_LINK1}">
+    <xacro:property name="LINK1" value="${MAX_LINK1}"/>
+  </xacro:if>
+  <xacro:if value="${MIN_LINK1 >= LINK1}">
+    <xacro:property name="LINK1" value="${MIN_LINK1}"/>
+  </xacro:if>
+  <xacro:if value="${LINK2 >= MAX_LINK2}">
+    <xacro:property name="LINK2" value="${MAX_LINK2}"/>
+  </xacro:if>
+  <xacro:if value="${MIN_LINK2 >= LINK2}">
+    <xacro:property name="LINK2" value="${MIN_LINK2}"/>
+  </xacro:if>
+  <xacro:if value="${LINK3 >= MAX_LINK3}">
+    <xacro:property name="LINK3" value="${MAX_LINK3}"/>
+  </xacro:if>
+  <xacro:if value="${MIN_LINK3 >= LINK3}">
+    <xacro:property name="LINK3" value="${MIN_LINK3}"/>
+  </xacro:if>
+  <xacro:if value="${LINK4 >= MAX_LINK4}">
+    <xacro:property name="LINK4" value="${MAX_LINK4}"/>
+  </xacro:if>
+  <xacro:if value="${MIN_LINK1 >= LINK4}">
+    <xacro:property name="LINK4" value="${MIN_LINK4}"/>
+  </xacro:if>
+  <xacro:if value="${LINK5 >= MAX_LINK5}">
+    <xacro:property name="LINK5" value="${MAX_LINK5}"/>
+  </xacro:if>
+  <xacro:if value="${MIN_LINK5 >= LINK5}">
+    <xacro:property name="LINK5" value="${MIN_LINK5}"/>
   </xacro:if>
   <xacro:property name="LINK1_LENGTH" value="${LINK1-0.045}"/>
@@ -60,5 +71,5 @@
   <link name="shelf">
     <visual>
-      <origin xyz="0 0.1 0" rpy="0 0 0"/>
+      <origin xyz="0 ${shelf_dist+0.1} 0" rpy="0 0 0"/>
       <geometry>
         <mesh filename="file:///$(find robot_description)/meshes/shelf.STL"/>
@@ -67,5 +78,5 @@
     </visual>
     <inertial>
-      <origin xyz="0 0.1 0" rpy="0 0 0"/>
+      <origin xyz="0 ${shelf_dist+0.1} 0" rpy="0 0 0"/>
       <mass value="5.0"/>
       <inertia
@@ -75,5 +86,5 @@
     </inertial>
     <collision>
-      <origin xyz="0 0.1 0" rpy="0 0 0"/>
+      <origin xyz="0 ${shelf_dist+0.1} 0" rpy="0 0 0"/>
       <geometry>
         <mesh filename="file:///$(find robot_description)/meshes/shelf.STL"/>
@@ -89,5 +100,5 @@
   <link name="obj1">
     <visual>
-      <origin xyz="-0.6 0.35 0.45" rpy="0 0 0"/>
+      <origin xyz="-0.6 ${shelf_dist+0.35} 0.45" rpy="0 0 0"/>
       <geometry>
         <cylinder radius="0.04" length="0.1"/>
@@ -96,5 +107,5 @@
     </visual>
     <inertial>
-      <origin xyz="-0.6 0.35 0.45" rpy="0 0 0"/>
+      <origin xyz="-0.6 ${shelf_dist+0.35} 0.45" rpy="0 0 0"/>
       <mass value="0.01"/>
       <inertia
@@ -104,5 +115,5 @@
     </inertial>
     <collision>
-      <origin xyz="-0.6 0.35 0.45" rpy="0 0 0"/>
+      <origin xyz="-0.6 ${shelf_dist+0.35} 0.45" rpy="0 0 0"/>
       <geometry>
         <cylinder radius="0.04" length="0.1"/>
@@ -116,5 +127,5 @@
   <link name="obj2">
     <visual>
-      <origin xyz="-0.3 0.35 0.45" rpy="0 0 0"/>
+      <origin xyz="-0.3 ${shelf_dist+0.35} 0.45" rpy="0 0 0"/>
       <geometry>
         <cylinder radius="0.04" length="0.1"/>
@@ -123,5 +134,5 @@
     </visual>
     <inertial>
-      <origin xyz="-0.3 0.35 0.45" rpy="0 0 0"/>
+      <origin xyz="-0.3 ${shelf_dist+0.35} 0.45" rpy="0 0 0"/>
       <mass value="0.01"/>
       <inertia
@@ -131,5 +142,5 @@
     </inertial>
     <collision>
-      <origin xyz="-0.3 0.35 0.45" rpy="0 0 0"/>
+      <origin xyz="-0.3 ${shelf_dist+0.35} 0.45" rpy="0 0 0"/>
       <geometry>
         <cylinder radius="0.04" length="0.1"/>
@@ -137,5 +148,5 @@
     </collision>
   </link>
-  <joint name="float_obj8" type="floating">
+  <joint name="float_obj8" type="fixed">
     <parent link="shelf"/>
     <child link="obj8"/>
@@ -143,5 +154,5 @@
   <link name="obj8">
     <visual>
-      <origin xyz="0.0 0.35 0.85" rpy="0 0 0"/>
+      <origin xyz="0.0 ${shelf_dist+0.35} 0.85" rpy="0 0 0"/>
       <geometry>
         <cylinder radius="0.04" length="0.1"/>
@@ -150,5 +161,5 @@
     </visual>
     <inertial>
-      <origin xyz="0.0 0.35 0.85" rpy="0 0 0"/>
+      <origin xyz="0.0 ${shelf_dist+0.35} 0.85" rpy="0 0 0"/>
       <mass value="0.01"/>
       <inertia
@@ -158,5 +169,5 @@
     </inertial>
     <collision>
-      <origin xyz="0.0 0.35 0.85" rpy="0 0 0"/>
+      <origin xyz="0.0 ${shelf_dist+0.35} 0.85" rpy="0 0 0"/>
       <geometry>
         <cylinder radius="0.04" length="0.1"/>
