Commit message: adjust fiction & damping

File: robot_description/urdf/parameter_v2.xacro (robot description, xacro)
@@ -2,5 +2,5 @@
 <robot name="robot" xmlns:xacro="http://www.ros.org/wiki/xacro">
   <xacro:property name="shelf_dist" value="0.2"/>
-  <xacro:property name="cylinder_obj_mass" value="2"/>
+  <xacro:property name="cylinder_obj_mass" value="0.01"/>
   <xacro:property name="params_path" value="$(find robot_description)/config/properties_v2.yaml"/>
   <xacro:property name="params" value="${xacro.load_yaml(params_path)}"/>
@@ -9,7 +9,7 @@
   <xacro:property name="LINK5" value="${params['link5_length']}"/>
   <xacro:property name="THETA_JOINT4" value="${params['theta_joint4']}"/>
-  <xacro:property name="MAX_LINK1" value="0.2"/>
-  <xacro:property name="MAX_LINK2" value="0.2"/>
-  <xacro:property name="MAX_LINK5" value="0.2"/>
+  <xacro:property name="MAX_LINK1" value="1.0"/>
+  <xacro:property name="MAX_LINK2" value="1.0"/>
+  <xacro:property name="MAX_LINK5" value="1.0"/>
   <xacro:property name="MIN_LINK1" value="0.045"/>
   <xacro:property name="MIN_LINK2" value="0.05125"/>

File: robot_description/urdf/robot_v2.xacro (robot description, xacro)
@@ -31,5 +31,5 @@
     <axis xyz="0 1 0"/>
     <limit lower="-0.40" upper="0.40" effort="0.0" velocity="0.0"/>
-    <dynamics damping="0" friction="1000"/>
+    <dynamics damping="0" friction="800"/>
   </joint>
   <link name="linkY">
@@ -49,5 +49,5 @@
     <axis xyz="0 0 1"/>
     <limit lower="-0.4" upper="0.4" effort="0.0" velocity="0.0"/>
-    <dynamics damping="0" friction="1000"/>
+    <dynamics damping="0" friction="600"/>
   </joint>
   <link name="link0">
@@ -80,5 +80,5 @@
     <axis xyz="0 0 1"/>
     <limit lower="-3.14" upper="3.14" effort="0.0" velocity="0.0"/>
-    <dynamics damping="0" friction="50"/>
+    <dynamics damping="0" friction="30"/>
   </joint>
   <link name="link1">
@@ -245,5 +245,5 @@
     <axis xyz="0 0 1"/>
     <limit lower="-1" upper="1" effort="0.0" velocity="0.0"/>
-    <dynamics damping="0" friction="5"/>
+    <dynamics damping="100" friction="30"/>
   </joint>
   <link name="link5">
@@ -276,5 +276,5 @@
     <axis xyz="0 0 1"/>
     <limit lower="-3.14" upper="3.14" effort="0.0" velocity="0.0"/>
-    <dynamics damping="0" friction="1.5"/>
+    <dynamics damping="100" friction="30"/>
   </joint>
   <link name="link_hook">

File: robot_description/urdf/spawn_obj.xacro (robot description, xacro)
@@ -435,4 +435,17 @@
   </link>
   <!-- next_floor -->
+  <!-- <gazebo>
+      <plugin name="gazebo_ros_joint_state_publisher"
+          filename="libgazebo_ros_joint_state_publisher.so">
+          <update_rate>20</update_rate>
+          <joint_name>float_obj1</joint_name>
+          <joint_name>float_obj2</joint_name>
+          <joint_name>float_obj3</joint_name>
+          <joint_name>float_obj4</joint_name>
+          <joint_name>float_obj5</joint_name>
+          <joint_name>float_obj6</joint_name>
+      </plugin>
+  </gazebo> -->
+  <!-- <xacro:include filename="$(find robot_description)/urdf/obj_gazebo.xacro"/> -->
   <gazebo reference="obj1">
     <material>Gazebo/Blue</material>
