Commit message: robot version2

File: robot_description/urdf/gazebo_v2.xacro (robot description, xacro)
@@ -6,11 +6,8 @@
           filename="libgazebo_ros_joint_state_publisher.so">
           <update_rate>20</update_rate>
-          <joint_name>joint0</joint_name>
+          <joint_name>jointX</joint_name>
+          <joint_name>jointY</joint_name>
+          <joint_name>jointZ</joint_name>
           <joint_name>joint1</joint_name>
-          <joint_name>joint2</joint_name>
-          <joint_name>joint3</joint_name>
-          <joint_name>joint4</joint_name>
-          <joint_name>joint5</joint_name>
-          <joint_name>joint6</joint_name>
       </plugin>
   </gazebo>
@@ -19,5 +16,23 @@
       <plugin>gazebo_ros2_control/GazeboSystem</plugin>
     </hardware>
-    <joint name="joint0">
+    <joint name="jointX">
+        <command_interface name="position">
+          <param name="min">-0.75</param>
+          <param name="max">0.75</param>
+        </command_interface>
+        <state_interface name="position">
+            <param name="initial_value">0.0</param>
+        </state_interface>
+    </joint>
+    <joint name="jointY">
+        <command_interface name="position">
+          <param name="min">-0.75</param>
+          <param name="max">0.75</param>
+        </command_interface>
+        <state_interface name="position">
+            <param name="initial_value">0.0</param>
+        </state_interface>
+    </joint>
+    <joint name="jointZ">
         <command_interface name="position">
           <param name="min">-0.75</param>
@@ -29,31 +44,4 @@
     </joint>
     <joint name="joint1">
-        <command_interface name="position">
-          <param name="min">-3.14</param>
-          <param name="max">3.14</param>
-        </command_interface>
-        <state_interface name="position">
-            <param name="initial_value">0.0</param>
-        </state_interface>
-    </joint>
-    <joint name="joint2">
-        <command_interface name="position">
-          <param name="min">-3.14</param>
-          <param name="max">3.14</param>
-        </command_interface>
-        <state_interface name="position">
-            <param name="initial_value">0.0</param>
-        </state_interface>
-    </joint>
-    <joint name="joint3">
-        <command_interface name="position">
-          <param name="min">-3.14</param>
-          <param name="max">3.14</param>
-        </command_interface>
-        <state_interface name="position">
-            <param name="initial_value">0.0</param>
-        </state_interface>
-    </joint>
-    <joint name="joint4">
         <command_interface name="position">
           <param name="min">-3.14</param>
@@ -85,5 +73,5 @@
   <gazebo>
     <plugin name="gazebo_ros2_control" filename="libgazebo_ros2_control.so">
-      <parameters>$(find robot_description)/config/controller.yaml</parameters>
+      <parameters>$(find robot_description)/config/controller_v2.yaml</parameters>
     </plugin>
   </gazebo>
@@ -100,7 +88,4 @@
   <gazebo reference="obj8">
     <material>Gazebo/Blue</material>
-  </gazebo>
-  <gazebo reference="link_slide">
-    <material>Gazebo/White</material>
   </gazebo>
   <gazebo reference="link0">
@@ -119,18 +104,6 @@
     <material>Gazebo/White</material>
   </gazebo>
-  <gazebo reference="link_joint3-1">
-    <material>Gazebo/Orange</material>
-  </gazebo>
-  <gazebo reference="link_joint3-2">
-    <material>Gazebo/Orange</material>
-  </gazebo>
-  <gazebo reference="link3">
-    <material>Gazebo/White</material>
-  </gazebo>
   <gazebo reference="link_joint4">
     <material>Gazebo/Orange</material>
-  </gazebo>
-  <gazebo reference="link4">
-    <material>Gazebo/White</material>
   </gazebo>
   <gazebo reference="link_joint5">

File: robot_description/urdf/parameter_v1.xacro (robot description, xacro)
@@ -1,5 +1,4 @@
 <?xml version="1.0"?>
 <robot name="robot" xmlns:xacro="http://www.ros.org/wiki/xacro">
-  <xacro:property name="PI" value="3.1415926535897931"/>
   <xacro:property name="shelf_dist" value="0.0"/>
   <xacro:property name="params_path" value="$(find robot_description)/config/properties.yaml"/>
@@ -10,4 +9,5 @@
   <xacro:property name="LINK4" value="${params['link4_length']}"/>
   <xacro:property name="LINK5" value="${params['link5_length']}"/>
+  <xacro:property name="THETA_JOINT4" value="${params['theta_joint4']}"/>
   <xacro:property name="MAX_LINK1" value="0.2"/>
   <xacro:property name="MAX_LINK2" value="0.2"/>
@@ -55,4 +55,5 @@
   <xacro:property name="LINK4_LENGTH" value="${LINK4-0.045}"/>
   <xacro:property name="LINK5_LENGTH" value="${LINK5+0.015}"/>
+  <xacro:property name="THETA_JOINT4_RAD" value="${pi*(THETA_JOINT4/180)}"/>
   <material name="orange">
     <color rgba="${255/255} ${108/255} ${10/255} 1.0"/>

File: robot_description/urdf/robot_v2.xacro (robot description, xacro)
@@ -2,43 +2,52 @@
 <robot name="robot" xmlns:xacro="http://www.ros.org/wiki/xacro">
   <!-- parameter -->
-  <xacro:include filename="$(find robot_description)/urdf/parameter.xacro"/>
+  <xacro:include filename="$(find robot_description)/urdf/parameter_v2.xacro"/>
   <link name="world"/>
   <!-- world -->
   <xacro:include filename="$(find robot_description)/urdf/world.xacro"/>
   <!-- robot -->
-  <joint name="fixed_robot" type="fixed">
+  <joint name="jointX" type="prismatic">
+    <origin xyz="0.0 0.0 0.2" rpy="0.0 0.0 0.0"/>
     <parent link="world"/>
-    <child link="link_slide"/>
-  </joint>
-  <link name="link_slide">
-    <visual>
-      <origin xyz="0 0 0" rpy="0 0 0"/>
-      <geometry>
-        <mesh filename="file:///$(find robot_description)/meshes/link_slide.STL"/>
-      </geometry>
-      <material name="white"/>
-    </visual>
-    <inertial>
-      <origin xyz="0 0 0" rpy="0 0 0"/>
-      <mass value="0.5"/>
-      <inertia
-        ixx="0.01" ixy="0.0" ixz="0.0"
-        iyy="0.01" iyz="0.0"
-        izz="0.01"/>
-    </inertial>
-    <collision>
-      <origin xyz="0 0 0" rpy="0 0 0"/>
-      <geometry>
-        <!-- <box size="1.0 0.2 0.2"/> -->
-        <mesh filename="file:///$(find robot_description)/meshes/link_slide.STL"/>
-      </geometry>
-    </collision>
-  </link>
-  <joint name="joint0" type="prismatic">
-    <origin xyz="0.0 0.0 0.2" rpy="0.0 0.0 0.0"/>
-    <parent link="link_slide"/>
-    <child link="link0"/>
+    <child link="linkX"/>
     <axis xyz="1 0 0"/>
     <limit lower="-0.40" upper="0.40" effort="0.0" velocity="0.0"/>
+    <dynamics damping="0" friction="1000"/>
+  </joint>
+  <link name="linkX">
+    <inertial>
+      <origin xyz="0 0 0" rpy="0 0 0"/>
+      <mass value="0.5"/>
+      <inertia
+        ixx="0.01" ixy="0.0" ixz="0.0"
+        iyy="0.01" iyz="0.0"
+        izz="0.01"/>
+    </inertial>
+  </link>
+  <joint name="jointY" type="prismatic">
+    <origin xyz="0.0 0.0 0.0" rpy="0.0 0.0 0.0"/>
+    <parent link="linkX"/>
+    <child link="linkY"/>
+    <axis xyz="0 1 0"/>
+    <limit lower="-0.40" upper="0.40" effort="0.0" velocity="0.0"/>
+    <dynamics damping="0" friction="1000"/>
+  </joint>
+  <link name="linkY">
+    <inertial>
+      <origin xyz="0 0 0" rpy="0 0 0"/>
+      <mass value="0.5"/>
+      <inertia
+        ixx="0.01" ixy="0.0" ixz="0.0"
+        iyy="0.01" iyz="0.0"
+        izz="0.01"/>
+    </inertial>
+  </link>
+  <joint name="jointZ" type="prismatic">
+    <origin xyz="0.0 0.0 0.0" rpy="0.0 0.0 0.0"/>
+    <parent link="linkY"/>
+    <child link="link0"/>
+    <axis xyz="0 0 1"/>
+    <limit lower="0" upper="0.40" effort="0.0" velocity="0.0"/>
+    <dynamics damping="0" friction="1000"/>
   </joint>
   <link name="link0">
@@ -65,5 +74,5 @@
     <axis xyz="0 0 1"/>
     <limit lower="-3.14" upper="3.14" effort="1000" velocity="1000"/>
-    <dynamics damping="0" friction="0"/>
+    <dynamics damping="0" friction="1000"/>
   </joint>
   <link name="link1">
@@ -105,15 +114,13 @@
     </inertial>
   </link>
-  <joint name="joint2" type="revolute">
+  <joint name="joint2" type="fixed">
     <parent link="link_joint2-1"/>
     <child link="link_joint2-2" />
     <origin rpy="${pi} ${pi/2} 0" xyz="0.04 0 ${LINK1_LENGTH+0.045}"/>
-    <axis xyz="0 0 1"/>
-    <limit lower="-3.14" upper="3.14" effort="1000" velocity="1000"/>
     <dynamics damping="0" friction="1000"/>
   </joint>
   <link name="link_joint2-2">
     <visual>
-      <origin xyz="0 0 -0.04" rpy="0 0 ${pi}"/>
+      <origin xyz="0 0 -0.04" rpy="0 0 ${pi+THETA_JOINT4_RAD}"/>
       <geometry>
         <mesh filename="file:///$(find robot_description)/meshes/joint_2-2.STL"/>
@@ -122,5 +129,5 @@
     </visual>
     <inertial>
-      <origin xyz="0 0 0.04" rpy="0 0 0"/>
+      <origin xyz="0 0 0.04" rpy="0 0 ${pi+THETA_JOINT4_RAD}"/>
       <mass value="0.01"/>
       <inertia
@@ -133,5 +140,5 @@
     <parent link="link_joint2-2"/>
     <child link="link2"/>
-    <origin rpy="0 ${-pi/2} ${-pi}" xyz="${(-LINK2_LENGTH/2)-0.085} 0 -0.04"/>
+    <origin rpy="0 ${-pi/2} ${-pi+THETA_JOINT4_RAD}" xyz="${(((-LINK2_LENGTH/2)-0.085)*sin((pi/2)-THETA_JOINT4_RAD))} ${((-LINK2_LENGTH/2)-0.085)*cos((pi/2)-THETA_JOINT4_RAD)} -0.04"/>
   </joint>
   <link name="link2">
@@ -152,14 +159,14 @@
     </inertial>
   </link>
-  <joint name="fixed_joint3-1" type="fixed">
+  <joint name="fixed_joint4" type="fixed">
     <parent link="link2"/>
-    <child link="link_joint3-1"/>
-    <origin rpy="0 ${pi/2} 0" xyz="0 0 ${-(LINK2_LENGTH/2)-0.005}"/>
-  </joint>
-  <link name="link_joint3-1">
-    <visual>
-      <origin xyz="0 0 0" rpy="0 0 0"/>
-      <geometry>
-        <mesh filename="file:///$(find robot_description)/meshes/joint_3-1.STL"/>
+    <child link="link_joint4"/>
+    <origin rpy="${pi} 0 0" xyz="0 0 ${(-LINK2_LENGTH/2)+0.04}"/>
+  </joint>
+  <link name="link_joint4">
+    <visual>
+      <origin xyz="0 0 0" rpy="0 0 0"/>
+      <geometry>
+        <mesh filename="file:///$(find robot_description)/meshes/joint_4.STL"/>
       </geometry>
       <material name="orange"/>
@@ -174,102 +181,8 @@
     </inertial>
   </link>
-  <joint name="joint3" type="revolute">
-    <parent link="link_joint3-1"/>
-    <child link="link_joint3-2" />
-    <origin rpy="${pi} ${pi} ${pi}" xyz="0 0 0.04"/>
-    <axis xyz="0 0 1"/>
-    <limit lower="-3.14" upper="3.14" effort="1000" velocity="1000"/>
-    <dynamics damping="0" friction="1000"/>
-  </joint>
-  <link name="link_joint3-2">
-    <visual>
-      <origin xyz="0 0 0.04" rpy="0 0 0"/>
-      <geometry>
-        <mesh filename="file:///$(find robot_description)/meshes/joint_3-2.STL"/>
-      </geometry>
-      <material name="orange"/>
-    </visual>
-    <inertial>
-      <origin xyz="0 0 0.04" rpy="0 0 0"/>
-      <mass value="0.01"/>
-      <inertia
-        ixx="0.01" ixy="0.0" ixz="0.0"
-        iyy="0.01" iyz="0.0"
-        izz="0.01"/>
-    </inertial>
-  </link>
-  <joint name="fixed_joint3-2" type="fixed">
-    <parent link="link_joint3-2"/>
-    <child link="link3"/>
-    <origin rpy="0 ${pi/2} 0" xyz="${(LINK3_LENGTH/2)+0.045} 0 0.04"/>
-  </joint>
-  <link name="link3">
-    <visual>
-      <origin xyz="0 0 0" rpy="0 0 0"/>
-      <geometry>
-        <cylinder radius="0.04" length="${LINK3_LENGTH}"/>
-      </geometry>
-      <material name="white"/>
-    </visual>
-    <inertial>
-      <origin xyz="0 0 0" rpy="0 0 0"/>
-      <mass value="0.01"/>
-      <inertia
-        ixx="0.01" ixy="0.0" ixz="0.0"
-        iyy="0.01" iyz="0.0"
-        izz="0.01"/>
-    </inertial>
-  </link>
-  <joint name="fixed_joint4" type="fixed">
-    <parent link="link3"/>
-    <child link="link_joint4"/>
-    <origin rpy="0 0 0" xyz="0 0 ${LINK3_LENGTH/2}"/>
-  </joint>
-  <link name="link_joint4">
-    <visual>
-      <origin xyz="0 0 0" rpy="0 0 0"/>
-      <geometry>
-        <mesh filename="file:///$(find robot_description)/meshes/joint_4.STL"/>
-      </geometry>
-      <material name="orange"/>
-    </visual>
-    <inertial>
-      <origin xyz="0 0 0" rpy="0 0 0"/>
-      <mass value="0.1"/>
-      <inertia
-        ixx="0.01" ixy="0.0" ixz="0.0"
-        iyy="0.01" iyz="0.0"
-        izz="0.01"/>
-    </inertial>
-  </link>
-  <joint name="joint4" type="revolute">
-    <parent link="link_joint4"/>
-    <child link="link4" />
-    <origin rpy="0 0 0" xyz="0 0 0.00625"/>
-    <axis xyz="0 0 1"/>
-    <limit lower="-3.14" upper="3.14" effort="1000" velocity="1000"/>
-    <dynamics damping="0" friction="1000"/>
-  </joint>
-  <link name="link4">
-    <visual>
-      <origin xyz="0 0 ${LINK4_LENGTH/2}" rpy="0 0 0"/>
-      <geometry>
-        <cylinder radius="0.035" length="${LINK4_LENGTH}"/>
-      </geometry>
-      <material name="white"/>
-    </visual>
-    <inertial>
-      <origin xyz="0 0 0" rpy="0 0 0"/>
-      <mass value="0.01"/>
-      <inertia
-        ixx="0.01" ixy="0.0" ixz="0.0"
-        iyy="0.01" iyz="0.0"
-        izz="0.01"/>
-    </inertial>
-  </link>
   <joint name="fixed_joint5" type="fixed">
-    <parent link="link4"/>
+    <parent link="link2"/>
     <child link="link_joint5"/>
-    <origin rpy="0 ${-pi/2} 0" xyz="0 0 ${LINK4_LENGTH+0.045}"/>
+    <origin rpy="0 ${pi/2} 0" xyz="0 0 ${(-LINK2_LENGTH/2)-0.005-0.00625}"/>
   </joint>
   <link name="link_joint5">
@@ -404,4 +317,4 @@
   </link>
   <!-- gazebo plugin -->
-  <xacro:include filename="$(find robot_description)/urdf/gazebo.xacro"/>
+  <xacro:include filename="$(find robot_description)/urdf/gazebo_v2.xacro"/>
 </robot>

Commit message: update robot2

File: robot_description/urdf/gazebo_v2.xacro (robot description, xacro)
@@ -36,6 +36,6 @@
     <joint name="jointZ">
         <command_interface name="position">
-          <param name="min">-0.75</param>
-          <param name="max">0.75</param>
+          <param name="min">0</param>
+          <param name="max">0.6</param>
         </command_interface>
         <state_interface name="position">

File: robot_description/urdf/parameter_v1.xacro (robot description, xacro)
@@ -2,5 +2,5 @@
 <robot name="robot" xmlns:xacro="http://www.ros.org/wiki/xacro">
   <xacro:property name="shelf_dist" value="0.0"/>
-  <xacro:property name="params_path" value="$(find robot_description)/config/properties.yaml"/>
+  <xacro:property name="params_path" value="$(find robot_description)/config/properties_v1.yaml"/>
   <xacro:property name="params" value="${xacro.load_yaml(params_path)}"/>
   <xacro:property name="LINK1" value="${params['link1_length']}"/>

File: robot_description/urdf/parameter_v2.xacro (robot description, xacro)
@@ -1,6 +1,6 @@
 <?xml version="1.0"?>
 <robot name="robot" xmlns:xacro="http://www.ros.org/wiki/xacro">
-  <xacro:property name="shelf_dist" value="0.5"/>
-  <xacro:property name="params_path" value="$(find robot_description)/config/properties.yaml"/>
+  <xacro:property name="shelf_dist" value="0.2"/>
+  <xacro:property name="params_path" value="$(find robot_description)/config/properties_v2.yaml"/>
   <xacro:property name="params" value="${xacro.load_yaml(params_path)}"/>
   <xacro:property name="LINK1" value="${params['link1_length']}"/>
@@ -12,5 +12,5 @@
   <xacro:property name="MAX_LINK5" value="0.2"/>
   <xacro:property name="MIN_LINK1" value="0.045"/>
-  <xacro:property name="MIN_LINK2" value="0.085"/>
+  <xacro:property name="MIN_LINK2" value="0.05125"/>
   <xacro:property name="MIN_LINK5" value="0.0115"/>
   <xacro:if value="${LINK1 >= MAX_LINK1}">

File: robot_description/urdf/robot_v2.xacro (robot description, xacro)
@@ -8,9 +8,9 @@
   <!-- robot -->
   <joint name="jointX" type="prismatic">
-    <origin xyz="0.0 0.0 0.2" rpy="0.0 0.0 0.0"/>
+    <origin xyz="0.0 0.0 0.4" rpy="0.0 0.0 0.0"/>
     <parent link="world"/>
     <child link="linkX"/>
     <axis xyz="1 0 0"/>
-    <limit lower="-0.40" upper="0.40" effort="0.0" velocity="0.0"/>
+    <limit lower="-0.60" upper="0.60" effort="0.0" velocity="0.0"/>
     <dynamics damping="0" friction="1000"/>
   </joint>
@@ -48,5 +48,5 @@
     <child link="link0"/>
     <axis xyz="0 0 1"/>
-    <limit lower="0" upper="0.40" effort="0.0" velocity="0.0"/>
+    <limit lower="-0.4" upper="0.4" effort="0.0" velocity="0.0"/>
     <dynamics damping="0" friction="1000"/>
   </joint>
@@ -252,65 +252,8 @@
         izz="0.01"/>
     </inertial>
-  </link>
-  <joint name="fixed_collision_box1" type="fixed">
-    <parent link="link_hook"/>
-    <child link="collision_box_1"/>
-    <origin rpy="0 0 0" xyz="0 0 0"/>
-  </joint>
-  <link name="collision_box_1">
-    <inertial>
-      <origin xyz="0 0 -0.0125" rpy="0 0 0"/>
-      <mass value="0.01"/>
-      <inertia
-        ixx="0.01" ixy="0.0" ixz="0.0"
-        iyy="0.01" iyz="0.0"
-        izz="0.01"/>
-    </inertial>
     <collision>
-      <origin xyz="0 0 -0.0125" rpy="0 0 0"/>
-      <geometry>
-        <box size="0.08 0.08 0.025"/>
-      </geometry>
-    </collision>
-  </link>
-  <joint name="fixed_collision_box2" type="fixed">
-    <parent link="collision_box_1"/>
-    <child link="collision_box_2"/>
-    <origin rpy="0 0 0" xyz="0 0 0"/>
-  </joint>
-  <link name="collision_box_2">
-    <inertial>
-      <origin xyz="-0.05 0 0.035" rpy="0 0 0"/>
-      <mass value="0.01"/>
-      <inertia
-        ixx="0.01" ixy="0.0" ixz="0.0"
-        iyy="0.01" iyz="0.0"
-        izz="0.01"/>
-    </inertial>
-    <collision>
-      <origin xyz="-0.05 0 0.035" rpy="0 0 0"/>
-      <geometry>
-        <box size="0.02 0.08 0.11"/>
-      </geometry>
-    </collision>
-  </link>
-  <joint name="fixed_collision_box3" type="fixed">
-    <parent link="collision_box_2"/>
-    <child link="collision_box_3"/>
-    <origin rpy="0 0 0" xyz="0 0 0"/>
-  </joint>
-  <link name="collision_box_3">
-    <inertial>
-      <origin xyz="-0.01 0 0.1" rpy="0 0 0"/>
-      <mass value="0.01"/>
-      <inertia
-        ixx="0.01" ixy="0.0" ixz="0.0"
-        iyy="0.01" iyz="0.0"
-        izz="0.01"/>
-    </inertial>
-    <collision>
-      <origin xyz="-0.01 0 0.1" rpy="0 0 0"/>
-      <geometry>
-        <box size="0.1 0.08 0.02"/>
+      <origin xyz="0.0 0.0 0.0" rpy="0.0 0.0 0.0"/>
+      <geometry>
+        <mesh filename="file:///$(find robot_description)/meshes/link_hook.STL"/>
       </geometry>
     </collision>

File: robot_description/urdf/world.xacro (robot description, xacro)
@@ -84,5 +84,5 @@
     </collision>
   </link>
-  <joint name="float_obj8" type="fixed">
+  <joint name="float_obj8" type="floating">
     <parent link="shelf"/>
     <child link="obj8"/>
@@ -90,5 +90,5 @@
   <link name="obj8">
     <visual>
-      <origin xyz="0.0 ${shelf_dist+0.35} 0.85" rpy="0 0 0"/>
+      <origin xyz="0.0 ${shelf_dist+0.35} 1.65" rpy="0 0 0"/>
       <geometry>
         <cylinder radius="0.04" length="0.1"/>
@@ -97,6 +97,6 @@
     </visual>
     <inertial>
-      <origin xyz="0.0 ${shelf_dist+0.35} 0.85" rpy="0 0 0"/>
-      <mass value="0.01"/>
+      <origin xyz="0.0 ${shelf_dist+0.35} 1.65" rpy="0 0 0"/>
+      <mass value="0.1"/>
       <inertia
         ixx="0.01" ixy="0.0" ixz="0.0"
@@ -105,5 +105,5 @@
     </inertial>
     <collision>
-      <origin xyz="0.0 ${shelf_dist+0.35} 0.85" rpy="0 0 0"/>
+      <origin xyz="0.0 ${shelf_dist+0.35} 1.65" rpy="0 0 0"/>
       <geometry>
         <cylinder radius="0.04" length="0.1"/>

Commit message: add velocity interface

File: robot_description/urdf/gazebo_v2.xacro (robot description, xacro)
@@ -10,4 +10,6 @@
           <joint_name>jointZ</joint_name>
           <joint_name>joint1</joint_name>
+          <joint_name>joint5</joint_name>
+          <joint_name>joint6</joint_name>
       </plugin>
   </gazebo>
@@ -21,4 +23,5 @@
           <param name="max">0.75</param>
         </command_interface>
+        <command_interface name="velocity"/>
         <state_interface name="position">
             <param name="initial_value">0.0</param>
@@ -30,4 +33,5 @@
           <param name="max">0.75</param>
         </command_interface>
+        <command_interface name="velocity"/>
         <state_interface name="position">
             <param name="initial_value">0.0</param>
@@ -39,4 +43,5 @@
           <param name="max">0.6</param>
         </command_interface>
+        <command_interface name="velocity"/>
         <state_interface name="position">
             <param name="initial_value">0.0</param>
@@ -48,4 +53,5 @@
           <param name="max">3.14</param>
         </command_interface>
+        <command_interface name="velocity"/>
         <state_interface name="position">
             <param name="initial_value">0.0</param>
@@ -57,4 +63,5 @@
           <param name="max">1</param>
         </command_interface>
+        <command_interface name="velocity"/>
         <state_interface name="position">
             <param name="initial_value">0.0</param>
@@ -66,4 +73,5 @@
           <param name="max">3.14</param>
         </command_interface>
+        <command_interface name="velocity"/>
         <state_interface name="position">
             <param name="initial_value">0.0</param>

File: robot_description/urdf/robot_v2.xacro (robot description, xacro)
@@ -73,5 +73,5 @@
     <origin rpy="0 0 0" xyz="0 0 0.04"/>
     <axis xyz="0 0 1"/>
-    <limit lower="-3.14" upper="3.14" effort="1000" velocity="1000"/>
+    <limit lower="-3.14" upper="3.14" effort="0.0" velocity="0.0"/>
     <dynamics damping="0" friction="1000"/>
   </joint>
@@ -208,5 +208,5 @@
     <origin rpy="0 0 0" xyz="0 0 0"/>
     <axis xyz="0 0 1"/>
-    <limit lower="-1" upper="1" effort="1000" velocity="1000"/>
+    <limit lower="-1" upper="1" effort="0.0" velocity="0.0"/>
     <dynamics damping="0" friction="1000"/>
   </joint>
@@ -233,5 +233,5 @@
     <origin rpy="0 ${pi/2} 0" xyz="${(LINK5_LENGTH)-0.015+0.0265} 0 0"/>
     <axis xyz="0 0 1"/>
-    <limit lower="-3.14" upper="3.14" effort="1000" velocity="1000"/>
+    <limit lower="-3.14" upper="3.14" effort="0.0" velocity="0.0"/>
     <dynamics damping="0" friction="1000"/>
   </joint>
