Commit message: update world

File: robot_description/urdf/gazebo_v2.xacro (robot description, xacro)
@@ -20,6 +20,6 @@
     <joint name="jointX">
         <command_interface name="position">
-          <param name="min">-0.75</param>
-          <param name="max">0.75</param>
+          <param name="min">-0.95</param>
+          <param name="max">0.95</param>
         </command_interface>
         <command_interface name="velocity"/>
@@ -85,7 +85,7 @@
   </gazebo>
   <!-- Base Link -->
-  <gazebo reference="shelf">
+  <!-- <gazebo reference="shelf">
     <material>Gazebo/White</material>
-  </gazebo>
+  </gazebo> -->
   <gazebo reference="obj1">
     <material>Gazebo/Blue</material>

File: robot_description/urdf/robot_v2.xacro (robot description, xacro)
@@ -5,5 +5,5 @@
   <link name="world"/>
   <!-- world -->
-  <xacro:include filename="$(find robot_description)/urdf/world.xacro"/>
+  <!-- <xacro:include filename="$(find robot_description)/urdf/world.xacro"/> -->
   <!-- robot -->
   <joint name="jointX" type="prismatic">
@@ -12,5 +12,5 @@
     <child link="linkX"/>
     <axis xyz="1 0 0"/>
-    <limit lower="-0.60" upper="0.60" effort="0.0" velocity="0.0"/>
+    <limit lower="-0.80" upper="0.80" effort="0.0" velocity="0.0"/>
     <dynamics damping="0" friction="1000"/>
   </joint>

File: robot_description/urdf/world.xacro (robot description, xacro)
@@ -1,4 +1,6 @@
 <?xml version="1.0"?>
-<robot name="robot" xmlns:xacro="http://www.ros.org/wiki/xacro">
+<robot name="world" xmlns:xacro="http://www.ros.org/wiki/xacro">
+  <xacro:include filename="$(find robot_description)/urdf/parameter_v2.xacro"/>
+  <link name="world"/>
   <joint name="fixed_shelf" type="fixed">
     <parent link="world"/>
@@ -28,86 +30,6 @@
     </collision>
   </link>
-  <joint name="float_obj1" type="floating">
-    <parent link="shelf"/>
-    <child link="obj1"/>
-    <dynamics damping="0.0" friction="10.0"/>
-    <limit effort="1" velocity="1.0" lower="-2.2" upper="0.7" />
-  </joint>
-  <link name="obj1">
-    <visual>
-      <origin xyz="-0.6 ${shelf_dist+0.35} 0.45" rpy="0 0 0"/>
-      <geometry>
-        <cylinder radius="0.04" length="0.1"/>
-      </geometry>
-      <material name="blue"/>
-    </visual>
-    <inertial>
-      <origin xyz="-0.6 ${shelf_dist+0.35} 0.45" rpy="0 0 0"/>
-      <mass value="0.01"/>
-      <inertia
-        ixx="0.01" ixy="0.0" ixz="0.0"
-        iyy="0.01" iyz="0.0"
-        izz="0.01"/>
-    </inertial>
-    <collision>
-      <origin xyz="-0.6 ${shelf_dist+0.35} 0.45" rpy="0 0 0"/>
-      <geometry>
-        <cylinder radius="0.04" length="0.1"/>
-      </geometry>
-    </collision>
-  </link>
-  <joint name="float_obj2" type="floating">
-    <parent link="shelf"/>
-    <child link="obj2"/>
-  </joint>
-  <link name="obj2">
-    <visual>
-      <origin xyz="-0.3 ${shelf_dist+0.35} 0.45" rpy="0 0 0"/>
-      <geometry>
-        <cylinder radius="0.04" length="0.1"/>
-      </geometry>
-      <material name="blue"/>
-    </visual>
-    <inertial>
-      <origin xyz="-0.3 ${shelf_dist+0.35} 0.45" rpy="0 0 0"/>
-      <mass value="0.01"/>
-      <inertia
-        ixx="0.01" ixy="0.0" ixz="0.0"
-        iyy="0.01" iyz="0.0"
-        izz="0.01"/>
-    </inertial>
-    <collision>
-      <origin xyz="-0.3 ${shelf_dist+0.35} 0.45" rpy="0 0 0"/>
-      <geometry>
-        <cylinder radius="0.04" length="0.1"/>
-      </geometry>
-    </collision>
-  </link>
-  <joint name="float_obj8" type="floating">
-    <parent link="shelf"/>
-    <child link="obj8"/>
-  </joint>
-  <link name="obj8">
-    <visual>
-      <origin xyz="0.0 ${shelf_dist+0.35} 1.65" rpy="0 0 0"/>
-      <geometry>
-        <cylinder radius="0.04" length="0.1"/>
-      </geometry>
-      <material name="blue"/>
-    </visual>
-    <inertial>
-      <origin xyz="0.0 ${shelf_dist+0.35} 1.65" rpy="0 0 0"/>
-      <mass value="0.1"/>
-      <inertia
-        ixx="0.01" ixy="0.0" ixz="0.0"
-        iyy="0.01" iyz="0.0"
-        izz="0.01"/>
-    </inertial>
-    <collision>
-      <origin xyz="0.0 ${shelf_dist+0.35} 1.65" rpy="0 0 0"/>
-      <geometry>
-        <cylinder radius="0.04" length="0.1"/>
-      </geometry>
-    </collision>
-  </link>
+  <gazebo reference="shelf">
+    <material>Gazebo/White</material>
+  </gazebo>
 </robot>

Commit message: add environment

File: robot_description/urdf/gazebo_v2.xacro (robot description, xacro)
@@ -85,15 +85,6 @@
   </gazebo>
   <!-- Base Link -->
-  <!-- <gazebo reference="shelf">
+  <gazebo reference="shelf">
     <material>Gazebo/White</material>
-  </gazebo> -->
-  <gazebo reference="obj1">
-    <material>Gazebo/Blue</material>
-  </gazebo>
-  <gazebo reference="obj2 ">
-    <material>Gazebo/Blue</material>
-  </gazebo>
-  <gazebo reference="obj8">
-    <material>Gazebo/Blue</material>
   </gazebo>
   <gazebo reference="link0">

File: robot_description/urdf/robot_v2.xacro (robot description, xacro)
@@ -5,5 +5,5 @@
   <link name="world"/>
   <!-- world -->
-  <!-- <xacro:include filename="$(find robot_description)/urdf/world.xacro"/> -->
+  <xacro:include filename="$(find robot_description)/urdf/world.xacro"/>
   <!-- robot -->
   <joint name="jointX" type="prismatic">
@@ -74,5 +74,5 @@
     <axis xyz="0 0 1"/>
     <limit lower="-3.14" upper="3.14" effort="0.0" velocity="0.0"/>
-    <dynamics damping="0" friction="1000"/>
+    <dynamics damping="0" friction="50"/>
   </joint>
   <link name="link1">
@@ -118,5 +118,5 @@
     <child link="link_joint2-2" />
     <origin rpy="${pi} ${pi/2} 0" xyz="0.04 0 ${LINK1_LENGTH+0.045}"/>
-    <dynamics damping="0" friction="1000"/>
+    <dynamics damping="0" friction="20"/>
   </joint>
   <link name="link_joint2-2">
@@ -209,5 +209,5 @@
     <axis xyz="0 0 1"/>
     <limit lower="-1" upper="1" effort="0.0" velocity="0.0"/>
-    <dynamics damping="0" friction="1000"/>
+    <dynamics damping="0" friction="5"/>
   </joint>
   <link name="link5">
@@ -234,5 +234,5 @@
     <axis xyz="0 0 1"/>
     <limit lower="-3.14" upper="3.14" effort="0.0" velocity="0.0"/>
-    <dynamics damping="0" friction="1000"/>
+    <dynamics damping="0" friction="1.5"/>
   </joint>
   <link name="link_hook">

File: robot_description/urdf/spawn_obj.xacro (robot description, xacro)
@@ -147,5 +147,5 @@
   </link>
   <!-- next_floor -->
-  <!-- <joint name="float_obj6" type="floating">
+  <joint name="float_obj6" type="floating">
     <parent link="world"/>
     <child link="obj6"/>
@@ -289,7 +289,7 @@
       </geometry>
     </collision>
-  </link> -->
+  </link>
   <!-- next_floor -->
-  <!-- <joint name="float_obj11" type="floating">
+  <joint name="float_obj11" type="floating">
     <parent link="world"/>
     <child link="obj11"/>
@@ -433,5 +433,5 @@
       </geometry>
     </collision>
-  </link> -->
+  </link>
   <!-- next_floor -->
   <gazebo reference="obj1">
@@ -450,5 +450,5 @@
     <material>Gazebo/Blue</material>
   </gazebo>
-  <!-- <gazebo reference="obj6">
+  <gazebo reference="obj6">
     <material>Gazebo/Blue</material>
   </gazebo>
@@ -479,4 +479,4 @@
   <gazebo reference="obj15">
     <material>Gazebo/Blue</material>
-  </gazebo> -->
+  </gazebo>
 </robot>

File: robot_description/urdf/world.xacro (robot description, xacro)
@@ -1,6 +1,6 @@
 <?xml version="1.0"?>
-<robot name="world" xmlns:xacro="http://www.ros.org/wiki/xacro">
-  <xacro:include filename="$(find robot_description)/urdf/parameter_v2.xacro"/>
-  <link name="world"/>
+<robot name="robot" xmlns:xacro="http://www.ros.org/wiki/xacro">
+  <!-- <xacro:include filename="$(find robot_description)/urdf/parameter_v2.xacro"/>
+  <link name="world"/> -->
   <joint name="fixed_shelf" type="fixed">
     <parent link="world"/>
@@ -30,6 +30,6 @@
     </collision>
   </link>
-  <gazebo reference="shelf">
+  <!-- <gazebo reference="shelf">
     <material>Gazebo/White</material>
-  </gazebo>
+  </gazebo> -->
 </robot>

Commit message: complete static world and object

File: robot_description/urdf/gazebo_v2.xacro (robot description, xacro)
@@ -85,7 +85,7 @@
   </gazebo>
   <!-- Base Link -->
-  <gazebo reference="shelf">
+  <!-- <gazebo reference="shelf">
     <material>Gazebo/White</material>
-  </gazebo>
+  </gazebo> -->
   <gazebo reference="link0">
     <material>Gazebo/White</material>

File: robot_description/urdf/parameter_v2.xacro (robot description, xacro)
@@ -2,4 +2,5 @@
 <robot name="robot" xmlns:xacro="http://www.ros.org/wiki/xacro">
   <xacro:property name="shelf_dist" value="0.2"/>
+  <xacro:property name="cylinder_obj_mass" value="2"/>
   <xacro:property name="params_path" value="$(find robot_description)/config/properties_v2.yaml"/>
   <xacro:property name="params" value="${xacro.load_yaml(params_path)}"/>

File: robot_description/urdf/robot_v2.xacro (robot description, xacro)
@@ -5,5 +5,5 @@
   <link name="world"/>
   <!-- world -->
-  <xacro:include filename="$(find robot_description)/urdf/world.xacro"/>
+  <!-- <xacro:include filename="$(find robot_description)/urdf/world.xacro"/> -->
   <!-- robot -->
   <joint name="jointX" type="prismatic">
@@ -67,4 +67,10 @@
         izz="0.01"/>
     </inertial>
+    <collision>
+      <origin xyz="0 0 0" rpy="0 0 0"/>
+      <geometry>
+        <mesh filename="file:///$(find robot_description)/meshes/link_base.STL"/>
+      </geometry>
+    </collision>
   </link>
   <joint name="joint1" type="revolute">
@@ -92,4 +98,10 @@
         izz="0.01"/>
     </inertial>
+    <collision>
+      <origin xyz="0 0 ${LINK1_LENGTH/2}" rpy="0 0 0"/>
+      <geometry>
+        <cylinder radius="0.04" length="${LINK1_LENGTH}"/>
+      </geometry>
+    </collision>
   </link>
   <joint name="fixed_link1" type="fixed">
@@ -136,4 +148,10 @@
         izz="0.01"/>
     </inertial>
+    <collision>
+      <origin xyz="0 0 -0.04" rpy="0 0 ${pi+THETA_JOINT4_RAD}"/>
+      <geometry>
+        <mesh filename="file:///$(find robot_description)/meshes/joint_2-2.STL"/>
+      </geometry>
+    </collision>
   </link>
   <joint name="fixed_joint2-2" type="fixed">
@@ -158,4 +176,10 @@
         izz="0.01"/>
     </inertial>
+    <collision>
+      <origin xyz="0 0 0.04" rpy="0 0 0"/>
+      <geometry>
+        <cylinder radius="0.04" length="${LINK2_LENGTH}"/>
+      </geometry>
+    </collision>
   </link>
   <joint name="fixed_joint4" type="fixed">
@@ -180,4 +204,10 @@
         izz="0.01"/>
     </inertial>
+    <collision>
+      <origin xyz="0 0 0" rpy="0 0 0"/>
+      <geometry>
+        <mesh filename="file:///$(find robot_description)/meshes/joint_4.STL"/>
+      </geometry>
+    </collision>
   </link>
   <joint name="fixed_joint5" type="fixed">
@@ -202,4 +232,10 @@
         izz="0.01"/>
     </inertial>
+    <collision>
+      <origin xyz="0 0 0" rpy="0 0 0"/>
+      <geometry>
+        <mesh filename="file:///$(find robot_description)/meshes/joint_5.STL"/>
+      </geometry>
+    </collision>
   </link>
   <joint name="joint5" type="revolute">
@@ -227,4 +263,10 @@
         izz="0.01"/>
     </inertial>
+    <collision>
+      <origin xyz="${(LINK5_LENGTH/2)-0.015} 0 0" rpy="0 ${pi/2} 0"/>
+      <geometry>
+        <cylinder radius="0.03" length="${LINK5_LENGTH}"/>
+      </geometry>
+    </collision>
   </link>
   <joint name="joint6" type="revolute">

File: robot_description/urdf/spawn_obj.xacro (robot description, xacro)
@@ -1,4 +1,4 @@
 <?xml version="1.0"?>
-<robot name="obj" xmlns:xacro="http://www.ros.org/wiki/xacro">
+<robot name="cylinder_object" xmlns:xacro="http://www.ros.org/wiki/xacro">
   <xacro:include filename="$(find robot_description)/urdf/parameter_v2.xacro"/>
   <link name="world"/>
@@ -19,5 +19,5 @@
     <inertial>
       <origin xyz="-0.6 ${shelf_dist+0.35} 0.45" rpy="0 0 0"/>
-      <mass value="0.01"/>
+      <mass value="${cylinder_obj_mass}"/>
       <inertia
         ixx="0.01" ixy="0.0" ixz="0.0"
@@ -46,5 +46,5 @@
     <inertial>
       <origin xyz="-0.3 ${shelf_dist+0.35} 0.45" rpy="0 0 0"/>
-      <mass value="0.01"/>
+      <mass value="${cylinder_obj_mass}"/>
       <inertia
         ixx="0.01" ixy="0.0" ixz="0.0"
@@ -75,5 +75,5 @@
     <inertial>
       <origin xyz="0.0 ${shelf_dist+0.35} 0.45" rpy="0 0 0"/>
-      <mass value="0.01"/>
+      <mass value="${cylinder_obj_mass}"/>
       <inertia
         ixx="0.01" ixy="0.0" ixz="0.0"
@@ -104,5 +104,5 @@
     <inertial>
       <origin xyz="0.3 ${shelf_dist+0.35} 0.45" rpy="0 0 0"/>
-      <mass value="0.01"/>
+      <mass value="${cylinder_obj_mass}"/>
       <inertia
         ixx="0.01" ixy="0.0" ixz="0.0"
@@ -133,5 +133,5 @@
     <inertial>
       <origin xyz="0.6 ${shelf_dist+0.35} 0.45" rpy="0 0 0"/>
-      <mass value="0.01"/>
+      <mass value="${cylinder_obj_mass}"/>
       <inertia
         ixx="0.01" ixy="0.0" ixz="0.0"
@@ -163,5 +163,5 @@
     <inertial>
       <origin xyz="-0.6 ${shelf_dist+0.35} 0.65" rpy="0 0 0"/>
-      <mass value="0.01"/>
+      <mass value="${cylinder_obj_mass}"/>
       <inertia
         ixx="0.01" ixy="0.0" ixz="0.0"
@@ -190,5 +190,5 @@
     <inertial>
       <origin xyz="-0.3 ${shelf_dist+0.35} 0.65" rpy="0 0 0"/>
-      <mass value="0.01"/>
+      <mass value="${cylinder_obj_mass}"/>
       <inertia
         ixx="0.01" ixy="0.0" ixz="0.0"
@@ -219,5 +219,5 @@
     <inertial>
       <origin xyz="0.0 ${shelf_dist+0.35} 0.65" rpy="0 0 0"/>
-      <mass value="0.01"/>
+      <mass value="${cylinder_obj_mass}"/>
       <inertia
         ixx="0.01" ixy="0.0" ixz="0.0"
@@ -248,5 +248,5 @@
     <inertial>
       <origin xyz="0.3 ${shelf_dist+0.35} 0.65" rpy="0 0 0"/>
-      <mass value="0.01"/>
+      <mass value="${cylinder_obj_mass}"/>
       <inertia
         ixx="0.01" ixy="0.0" ixz="0.0"
@@ -277,5 +277,5 @@
     <inertial>
       <origin xyz="0.6 ${shelf_dist+0.35} 0.65" rpy="0 0 0"/>
-      <mass value="0.01"/>
+      <mass value="${cylinder_obj_mass}"/>
       <inertia
         ixx="0.01" ixy="0.0" ixz="0.0"
@@ -307,5 +307,5 @@
     <inertial>
       <origin xyz="-0.6 ${shelf_dist+0.35} 0.85" rpy="0 0 0"/>
-      <mass value="0.01"/>
+      <mass value="${cylinder_obj_mass}"/>
       <inertia
         ixx="0.01" ixy="0.0" ixz="0.0"
@@ -334,5 +334,5 @@
     <inertial>
       <origin xyz="-0.3 ${shelf_dist+0.35} 0.85" rpy="0 0 0"/>
-      <mass value="0.01"/>
+      <mass value="${cylinder_obj_mass}"/>
       <inertia
         ixx="0.01" ixy="0.0" ixz="0.0"
@@ -363,5 +363,5 @@
     <inertial>
       <origin xyz="0.0 ${shelf_dist+0.35} 0.85" rpy="0 0 0"/>
-      <mass value="0.01"/>
+      <mass value="${cylinder_obj_mass}"/>
       <inertia
         ixx="0.01" ixy="0.0" ixz="0.0"
@@ -392,5 +392,5 @@
     <inertial>
       <origin xyz="0.3 ${shelf_dist+0.35} 0.85" rpy="0 0 0"/>
-      <mass value="0.01"/>
+      <mass value="${cylinder_obj_mass}"/>
       <inertia
         ixx="0.01" ixy="0.0" ixz="0.0"
@@ -421,5 +421,5 @@
     <inertial>
       <origin xyz="0.6 ${shelf_dist+0.35} 0.85" rpy="0 0 0"/>
-      <mass value="0.01"/>
+      <mass value="${cylinder_obj_mass}"/>
       <inertia
         ixx="0.01" ixy="0.0" ixz="0.0"

File: robot_description/urdf/world.xacro (robot description, xacro)
@@ -1,6 +1,6 @@
 <?xml version="1.0"?>
-<robot name="robot" xmlns:xacro="http://www.ros.org/wiki/xacro">
-  <!-- <xacro:include filename="$(find robot_description)/urdf/parameter_v2.xacro"/>
-  <link name="world"/> -->
+<robot name="environment" xmlns:xacro="http://www.ros.org/wiki/xacro">
+  <xacro:include filename="$(find robot_description)/urdf/parameter_v2.xacro"/>
+  <link name="world"/>
   <joint name="fixed_shelf" type="fixed">
     <parent link="world"/>
@@ -30,6 +30,6 @@
     </collision>
   </link>
-  <!-- <gazebo reference="shelf">
+  <gazebo reference="shelf">
     <material>Gazebo/White</material>
-  </gazebo> -->
+  </gazebo>
 </robot>

Commit message: add end effector

File: robot_description/urdf/gazebo_v2.xacro (robot description, xacro)
@@ -112,5 +112,5 @@
     <material>Gazebo/White</material>
   </gazebo>
-  <gazebo reference="link_hook">
+  <gazebo reference="end_effector">
     <material>Gazebo/Orange</material>
   </gazebo>

File: robot_description/urdf/obj_gazebo.xacro (robot description, xacro)
@@ -3,13 +3,13 @@
   <!-- gazebo plugin -->
   <gazebo>
-      <plugin name="gazebo_ros_joint_state_publisher"
+      <plugin name="gazebo_ros_joint_state_publisher_obj"
           filename="libgazebo_ros_joint_state_publisher.so">
           <update_rate>20</update_rate>
           <joint_name>float_obj1</joint_name>
-          <joint_name>float_obj2</joint_name>
+          <!-- <joint_name>float_obj2</joint_name>
           <joint_name>float_obj3</joint_name>
           <joint_name>float_obj4</joint_name>
           <joint_name>float_obj5</joint_name>
-          <joint_name>float_obj6</joint_name>
+          <joint_name>float_obj6</joint_name> -->
       </plugin>
   </gazebo>
@@ -19,8 +19,12 @@
     </hardware>
     <joint name="float_obj1">
+        <command_interface name="position">
+          <!-- <param name="min">-5.0</param>
+          <param name="max">5.0</param> -->
+        </command_interface>
         <state_interface name="position">
         </state_interface>
     </joint>
-    <joint name="float_obj2">
+    <!-- <joint name="float_obj2">
         <state_interface name="position">
         </state_interface>
@@ -41,5 +45,10 @@
         <state_interface name="position">
         </state_interface>
-    </joint>
+    </joint> -->
   </ros2_control>
+  <gazebo>
+    <plugin name="gazebo_ros2_control_obj" filename="libgazebo_ros2_control.so">
+      <parameters>$(find robot_description)/config/controller_obj.yaml</parameters>
+    </plugin>
+  </gazebo>
 </robot>

File: robot_description/urdf/robot_v2.xacro (robot description, xacro)
@@ -272,5 +272,5 @@
   <joint name="joint6" type="revolute">
     <parent link="link5"/>
-    <child link="link_hook" />
+    <child link="end_effector" />
     <origin rpy="0 ${pi/2} 0" xyz="${(LINK5_LENGTH)-0.015+0.0265} 0 0"/>
     <axis xyz="0 0 1"/>
@@ -278,9 +278,9 @@
     <dynamics damping="100" friction="30"/>
   </joint>
-  <link name="link_hook">
-    <visual>
-      <origin xyz="0 0 0" rpy="0 0 0"/>
-      <geometry>
-        <mesh filename="file:///$(find robot_description)/meshes/link_hook.STL"/>
+  <link name="end_effector">
+    <visual>
+      <origin xyz="0 0 0" rpy="0 0 0"/>
+      <geometry>
+        <mesh filename="file:///$(find robot_description)/meshes/end_effectorL.STL"/>
       </geometry>
       <material name="orange"/>
@@ -297,5 +297,5 @@
       <origin xyz="0.0 0.0 0.0" rpy="0.0 0.0 0.0"/>
       <geometry>
-        <mesh filename="file:///$(find robot_description)/meshes/link_hook.STL"/>
+        <mesh filename="file:///$(find robot_description)/meshes/end_effectorL.STL"/>
       </geometry>
     </collision>

File: robot_description/urdf/spawn_obj.xacro (robot description, xacro)
@@ -351,5 +351,5 @@
     <child link="obj13"/>
     <dynamics damping="0.0" friction="10.0"/>
-    <limit effort="1" velocity="1.0" lower="-2.2" upper="0.7" />
+    <limit effort="1" velocity="1.0" lower="-5.0" upper="5.0" />
   </joint>
   <link name="obj13">
@@ -435,16 +435,4 @@
   </link>
   <!-- next_floor -->
-  <!-- <gazebo>
-      <plugin name="gazebo_ros_joint_state_publisher"
-          filename="libgazebo_ros_joint_state_publisher.so">
-          <update_rate>20</update_rate>
-          <joint_name>float_obj1</joint_name>
-          <joint_name>float_obj2</joint_name>
-          <joint_name>float_obj3</joint_name>
-          <joint_name>float_obj4</joint_name>
-          <joint_name>float_obj5</joint_name>
-          <joint_name>float_obj6</joint_name>
-      </plugin>
-  </gazebo> -->
   <!-- <xacro:include filename="$(find robot_description)/urdf/obj_gazebo.xacro"/> -->
   <gazebo reference="obj1">
