Commit message: test ws

File: robot_description/urdf/spawn_obj.xacro (robot description, xacro)
@@ -6,6 +6,7 @@
     <parent link="world"/>
     <child link="obj1"/>
-    <dynamics damping="0.0" friction="10.0"/>
-    <limit effort="1" velocity="1.0" lower="-2.2" upper="0.7" />
+    <!-- <origin xyz="0.0 0.0 0.0" rpy="0.0 0.0 0.0"/>
+    <axis xyz="0 1 0"/>
+    <limit lower="-0.40" upper="0.40" effort="0.0" velocity="0.0"/> -->
   </joint>
   <link name="obj1">
