Commit message: test script shell

File: robot_description/urdf/obj_gazebo.xacro (robot description, xacro)
@@ -14,5 +14,5 @@
       </plugin>
   </gazebo>
-  <ros2_control name="GazeboSystem" type="system">
+  <ros2_control name="GazeboSystem_obj" type="system">
     <hardware>
       <plugin>gazebo_ros2_control/GazeboSystem</plugin>
@@ -20,7 +20,8 @@
     <joint name="float_obj1">
         <command_interface name="position">
-          <!-- <param name="min">-5.0</param>
-          <param name="max">5.0</param> -->
+          <param name="min">-5.0</param>
+          <param name="max">5.0</param>
         </command_interface>
+        <command_interface name="velocity"/>
         <state_interface name="position">
         </state_interface>

File: robot_description/urdf/robot_v2.xacro (robot description, xacro)
@@ -282,5 +282,5 @@
       <origin xyz="0 0 0" rpy="0 0 0"/>
       <geometry>
-        <mesh filename="file:///$(find robot_description)/meshes/end_effectorL.STL"/>
+        <mesh filename="file:///$(find robot_description)/meshes/end_effectorI.STL"/>
       </geometry>
       <material name="orange"/>
@@ -297,5 +297,5 @@
       <origin xyz="0.0 0.0 0.0" rpy="0.0 0.0 0.0"/>
       <geometry>
-        <mesh filename="file:///$(find robot_description)/meshes/end_effectorL.STL"/>
+        <mesh filename="file:///$(find robot_description)/meshes/end_effectorI.STL"/>
       </geometry>
     </collision>

File: robot_description/urdf/world.xacro (robot description, xacro)
@@ -17,5 +17,5 @@
     <inertial>
       <origin xyz="0 ${shelf_dist+0.1} 0" rpy="0 0 0"/>
-      <mass value="5.0"/>
+      <mass value="1000.0"/>
       <inertia
         ixx="0.01" ixy="0.0" ixz="0.0"

Commit message: game logic & scoring node

File: robot_description/urdf/obj_gazebo.xacro (robot description, xacro)
@@ -2,54 +2,76 @@
 <robot xmlns:xacro="http://www.ros.org/wiki/xacro">
   <!-- gazebo plugin -->
+  <xacro:macro name="cylider_gazebo" params="name_obj">
+    <joint_name>${name_obj}_prisX</joint_name>
+    <joint_name>${name_obj}_prisY</joint_name>
+    <joint_name>${name_obj}_prisZ</joint_name>
+    <joint_name>${name_obj}_revolX</joint_name>
+    <joint_name>${name_obj}_revolY</joint_name>
+    <joint_name>${name_obj}_revolZ</joint_name>
+  </xacro:macro>
   <gazebo>
       <plugin name="gazebo_ros_joint_state_publisher_obj"
           filename="libgazebo_ros_joint_state_publisher.so">
-          <update_rate>20</update_rate>
-          <joint_name>float_obj1</joint_name>
-          <!-- <joint_name>float_obj2</joint_name>
-          <joint_name>float_obj3</joint_name>
-          <joint_name>float_obj4</joint_name>
-          <joint_name>float_obj5</joint_name>
-          <joint_name>float_obj6</joint_name> -->
+          <xacro:cylider_gazebo name_obj="obj1"/>
+          <xacro:cylider_gazebo name_obj="obj2"/>
+          <xacro:cylider_gazebo name_obj="obj3"/>
+          <xacro:cylider_gazebo name_obj="obj4"/>
+          <xacro:cylider_gazebo name_obj="obj5"/>
+          <xacro:cylider_gazebo name_obj="obj6"/>
+          <xacro:cylider_gazebo name_obj="obj7"/>
+          <xacro:cylider_gazebo name_obj="obj8"/>
+          <xacro:cylider_gazebo name_obj="obj9"/>
+          <xacro:cylider_gazebo name_obj="obj10"/>
+          <xacro:cylider_gazebo name_obj="obj11"/>
+          <xacro:cylider_gazebo name_obj="obj12"/>
+          <xacro:cylider_gazebo name_obj="obj13"/>
+          <xacro:cylider_gazebo name_obj="obj14"/>
+          <xacro:cylider_gazebo name_obj="obj15"/>
       </plugin>
   </gazebo>
-  <ros2_control name="GazeboSystem_obj" type="system">
-    <hardware>
-      <plugin>gazebo_ros2_control/GazeboSystem</plugin>
-    </hardware>
-    <joint name="float_obj1">
-        <command_interface name="position">
-          <param name="min">-5.0</param>
-          <param name="max">5.0</param>
-        </command_interface>
-        <command_interface name="velocity"/>
-        <state_interface name="position">
-        </state_interface>
-    </joint>
-    <!-- <joint name="float_obj2">
-        <state_interface name="position">
-        </state_interface>
-    </joint>
-    <joint name="float_obj3">
-        <state_interface name="position">
-        </state_interface>
-    </joint>
-    <joint name="float_obj4">
-        <state_interface name="position">
-        </state_interface>
-    </joint>
-    <joint name="float_obj5">
-        <state_interface name="position">
-        </state_interface>
-    </joint>
-    <joint name="float_obj6">
-        <state_interface name="position">
-        </state_interface>
-    </joint> -->
-  </ros2_control>
-  <gazebo>
-    <plugin name="gazebo_ros2_control_obj" filename="libgazebo_ros2_control.so">
-      <parameters>$(find robot_description)/config/controller_obj.yaml</parameters>
-    </plugin>
+  <gazebo reference="obj1">
+    <material>Gazebo/Blue</material>
+  </gazebo>
+  <gazebo reference="obj2">
+    <material>Gazebo/Blue</material>
+  </gazebo>
+  <gazebo reference="obj3">
+    <material>Gazebo/Blue</material>
+  </gazebo>
+  <gazebo reference="obj4">
+    <material>Gazebo/Blue</material>
+  </gazebo>
+  <gazebo reference="obj5">
+    <material>Gazebo/Blue</material>
+  </gazebo>
+  <gazebo reference="obj6">
+    <material>Gazebo/Blue</material>
+  </gazebo>
+  <gazebo reference="obj7">
+    <material>Gazebo/Blue</material>
+  </gazebo>
+  <gazebo reference="obj8">
+    <material>Gazebo/Blue</material>
+  </gazebo>
+  <gazebo reference="obj9">
+    <material>Gazebo/Blue</material>
+  </gazebo>
+  <gazebo reference="obj10">
+    <material>Gazebo/Blue</material>
+  </gazebo>
+  <gazebo reference="obj11">
+    <material>Gazebo/Blue</material>
+  </gazebo>
+  <gazebo reference="obj12">
+    <material>Gazebo/Blue</material>
+  </gazebo>
+  <gazebo reference="obj13">
+    <material>Gazebo/Blue</material>
+  </gazebo>
+  <gazebo reference="obj14">
+    <material>Gazebo/Blue</material>
+  </gazebo>
+  <gazebo reference="obj15">
+    <material>Gazebo/Blue</material>
   </gazebo>
 </robot>
