Commit message: Update

File: robot_description/urdf/cylinder_obj.xacro (robot description, xacro)
@@ -2,4 +2,7 @@
 <robot name="cylinder_object" xmlns:xacro="http://www.ros.org/wiki/xacro">
   <xacro:include filename="$(find robot_description)/urdf/parameter.xacro"/>
+  <xacro:property name="IXX" value="${((cylinder_obj_mass*0.04*0.04)/4)+((cylinder_obj_mass*0.1*0.1)/12)}"/>
+  <xacro:property name="IYY" value="${((cylinder_obj_mass*0.04*0.04)/4)+((cylinder_obj_mass*0.1*0.1)/12)}"/>
+  <xacro:property name="IZZ" value="${(cylinder_obj_mass*0.04*0.04)/2}"/>
   <link name="world"/>
   <xacro:macro name="cylinder_obj" params="name_obj dist_x dist_z">
@@ -114,7 +117,7 @@
             <mass value="${cylinder_obj_mass}"/>
             <inertia
-                ixx="0.01" ixy="0.0" ixz="0.0"
-                iyy="0.01" iyz="0.0"
-                izz="0.01"/>
+                ixx="${IXX}" ixy="0.0" ixz="0.0"
+                iyy="${IYY}" iyz="0.0"
+                izz="${IZZ}"/>
         </inertial>
         <collision>

File: robot_description/urdf/gazebo.xacro (robot description, xacro)
@@ -103,5 +103,5 @@
     <material>Gazebo/Orange</material>
   </gazebo>
-  <gazebo reference="link5">
+  <gazebo reference="link3">
     <material>Gazebo/White</material>
   </gazebo>

File: robot_description/urdf/parameter.xacro (robot description, xacro)
@@ -7,12 +7,12 @@
   <xacro:property name="LINK1" value="${params['link1_length']}"/>
   <xacro:property name="LINK2" value="${params['link2_length']}"/>
-  <xacro:property name="LINK5" value="${params['link5_length']}"/>
-  <xacro:property name="THETA_JOINT4" value="${params['theta_joint4']}"/>
+  <xacro:property name="LINK3" value="${params['link3_length']}"/>
+  <xacro:property name="THETA_JOINT2" value="${params['theta_joint2']}"/>
   <xacro:property name="MAX_LINK1" value="1.0"/>
   <xacro:property name="MAX_LINK2" value="1.0"/>
-  <xacro:property name="MAX_LINK5" value="1.0"/>
+  <xacro:property name="MAX_LINK3" value="1.0"/>
   <xacro:property name="MIN_LINK1" value="0.045"/>
   <xacro:property name="MIN_LINK2" value="0.05125"/>
-  <xacro:property name="MIN_LINK5" value="0.0115"/>
+  <xacro:property name="MIN_LINK3" value="0.0115"/>
   <xacro:if value="${LINK1 >= MAX_LINK1}">
     <xacro:property name="LINK1" value="${MAX_LINK1}"/>
@@ -27,14 +27,14 @@
     <xacro:property name="LINK2" value="${MIN_LINK2}"/>
   </xacro:if>
-  <xacro:if value="${LINK5 >= MAX_LINK5}">
-    <xacro:property name="LINK5" value="${MAX_LINK5}"/>
+  <xacro:if value="${LINK3 >= MAX_LINK3}">
+    <xacro:property name="LINK3" value="${MAX_LINK3}"/>
   </xacro:if>
-  <xacro:if value="${MIN_LINK5 >= LINK5}">
-    <xacro:property name="LINK5" value="${MIN_LINK5}"/>
+  <xacro:if value="${MIN_LINK3 >= LINK3}">
+    <xacro:property name="LINK3" value="${MIN_LINK3}"/>
   </xacro:if>
   <xacro:property name="LINK1_LENGTH" value="${LINK1-0.045}"/>
   <xacro:property name="LINK2_LENGTH" value="${LINK2-0.045-0.00625}"/>
-  <xacro:property name="LINK5_LENGTH" value="${LINK5+0.015}"/>
-  <xacro:property name="THETA_JOINT4_RAD" value="${pi*(THETA_JOINT4/180)}"/>
+  <xacro:property name="LINK3_LENGTH" value="${LINK3+0.015}"/>
+  <xacro:property name="THETA_JOINT2_RAD" value="${pi*(THETA_JOINT2/180)}"/>
   <material name="orange">
     <color rgba="${255/255} ${108/255} ${10/255} 1.0"/>

File: robot_description/urdf/robot.xacro (robot description, xacro)
@@ -134,5 +134,5 @@
   <link name="link_joint2-2">
     <visual>
-      <origin xyz="0 0 -0.04" rpy="0 0 ${pi+THETA_JOINT4_RAD}"/>
+      <origin xyz="0 0 -0.04" rpy="0 0 ${pi+THETA_JOINT2_RAD}"/>
       <geometry>
         <mesh filename="file:///$(find robot_description)/meshes/joint_2-2.STL"/>
@@ -141,5 +141,5 @@
     </visual>
     <inertial>
-      <origin xyz="0 0 0.04" rpy="0 0 ${pi+THETA_JOINT4_RAD}"/>
+      <origin xyz="0 0 0.04" rpy="0 0 ${pi+THETA_JOINT2_RAD}"/>
       <mass value="0.01"/>
       <inertia
@@ -149,5 +149,5 @@
     </inertial>
     <collision>
-      <origin xyz="0 0 -0.04" rpy="0 0 ${pi+THETA_JOINT4_RAD}"/>
+      <origin xyz="0 0 -0.04" rpy="0 0 ${pi+THETA_JOINT2_RAD}"/>
       <geometry>
         <mesh filename="file:///$(find robot_description)/meshes/joint_2-2.STL"/>
@@ -158,5 +158,5 @@
     <parent link="link_joint2-2"/>
     <child link="link2"/>
-    <origin rpy="0 ${-pi/2} ${-pi+THETA_JOINT4_RAD}" xyz="${(((-LINK2_LENGTH/2)-0.085)*sin((pi/2)-THETA_JOINT4_RAD))} ${((-LINK2_LENGTH/2)-0.085)*cos((pi/2)-THETA_JOINT4_RAD)} -0.04"/>
+    <origin rpy="0 ${-pi/2} ${-pi+THETA_JOINT2_RAD}" xyz="${(((-LINK2_LENGTH/2)-0.085)*sin((pi/2)-THETA_JOINT2_RAD))} ${((-LINK2_LENGTH/2)-0.085)*cos((pi/2)-THETA_JOINT2_RAD)} -0.04"/>
   </joint>
   <link name="link2">
@@ -241,5 +241,5 @@
   <joint name="joint5" type="revolute">
     <parent link="link_joint5"/>
-    <child link="link5" />
+    <child link="link3" />
     <origin rpy="0 0 0" xyz="0 0 0"/>
     <axis xyz="0 0 1"/>
@@ -247,9 +247,9 @@
     <dynamics damping="100" friction="30"/>
   </joint>
-  <link name="link5">
-    <visual>
-      <origin xyz="${(LINK5_LENGTH/2)-0.015} 0 0" rpy="0 ${pi/2} 0"/>
-      <geometry>
-        <cylinder radius="0.03" length="${LINK5_LENGTH}"/>
+  <link name="link3">
+    <visual>
+      <origin xyz="${(LINK3_LENGTH/2)-0.015} 0 0" rpy="0 ${pi/2} 0"/>
+      <geometry>
+        <cylinder radius="0.03" length="${LINK3_LENGTH}"/>
       </geometry>
       <material name="white"/>
@@ -264,14 +264,14 @@
     </inertial>
     <collision>
-      <origin xyz="${(LINK5_LENGTH/2)-0.015} 0 0" rpy="0 ${pi/2} 0"/>
-      <geometry>
-        <cylinder radius="0.03" length="${LINK5_LENGTH}"/>
+      <origin xyz="${(LINK3_LENGTH/2)-0.015} 0 0" rpy="0 ${pi/2} 0"/>
+      <geometry>
+        <cylinder radius="0.03" length="${LINK3_LENGTH}"/>
       </geometry>
     </collision>
   </link>
   <joint name="joint6" type="revolute">
-    <parent link="link5"/>
+    <parent link="link3"/>
     <child link="end_effector" />
-    <origin rpy="0 ${pi/2} 0" xyz="${(LINK5_LENGTH)-0.015+0.0265} 0 0"/>
+    <origin rpy="0 ${pi/2} 0" xyz="${(LINK3_LENGTH)-0.015+0.0265} 0 0"/>
     <axis xyz="0 0 1"/>
     <limit lower="-3.14" upper="3.14" effort="0.0" velocity="0.0"/>

Commit message: add color & timeout status

File: robot_description/urdf/cylinder_obj.xacro (robot description, xacro)
@@ -6,5 +6,5 @@
   <xacro:property name="IZZ" value="${(cylinder_obj_mass*0.04*0.04)/2}"/>
   <link name="world"/>
-  <xacro:macro name="cylinder_obj" params="name_obj dist_x dist_z">
+  <xacro:macro name="cylinder_obj" params="name_obj dist_x dist_z color">
     <joint name="${name_obj}_prisX" type="prismatic">
         <origin xyz="${dist_x} ${shelf_dist+0.35} ${dist_z}" rpy="0.0 0.0 0.0"/>
@@ -111,5 +111,5 @@
                 <cylinder radius="0.04" length="0.1"/>
             </geometry>
-            <material name="blue"/>
+            <material name="${color}"/>
         </visual>
         <inertial>
@@ -129,19 +129,19 @@
     </link>
   </xacro:macro>
-  <xacro:cylinder_obj name_obj="obj1" dist_x="-0.6" dist_z="0.45"/>
-  <xacro:cylinder_obj name_obj="obj2" dist_x="-0.3" dist_z="0.45"/>
-  <xacro:cylinder_obj name_obj="obj3" dist_x="0.0" dist_z="0.45"/>
-  <xacro:cylinder_obj name_obj="obj4" dist_x="0.3" dist_z="0.45"/>
-  <xacro:cylinder_obj name_obj="obj5" dist_x="0.6" dist_z="0.45"/>
-  <xacro:cylinder_obj name_obj="obj6" dist_x="-0.6" dist_z="0.65"/>
-  <xacro:cylinder_obj name_obj="obj7" dist_x="-0.3" dist_z="0.65"/>
-  <xacro:cylinder_obj name_obj="obj8" dist_x="0.0" dist_z="0.65"/>
-  <xacro:cylinder_obj name_obj="obj9" dist_x="0.3" dist_z="0.65"/>
-  <xacro:cylinder_obj name_obj="obj10" dist_x="0.6" dist_z="0.65"/>
-  <xacro:cylinder_obj name_obj="obj11" dist_x="-0.6" dist_z="0.85"/>
-  <xacro:cylinder_obj name_obj="obj12" dist_x="-0.3" dist_z="0.85"/>
-  <xacro:cylinder_obj name_obj="obj13" dist_x="0.0" dist_z="0.85"/>
-  <xacro:cylinder_obj name_obj="obj14" dist_x="0.3" dist_z="0.85"/>
-  <xacro:cylinder_obj name_obj="obj15" dist_x="0.6" dist_z="0.85"/>
+  <xacro:cylinder_obj name_obj="obj1" dist_x="-0.6" dist_z="0.45" color="green"/>
+  <xacro:cylinder_obj name_obj="obj2" dist_x="-0.3" dist_z="0.45" color="green"/>
+  <xacro:cylinder_obj name_obj="obj3" dist_x="0.0" dist_z="0.45" color="green"/>
+  <xacro:cylinder_obj name_obj="obj4" dist_x="0.3" dist_z="0.45" color="green"/>
+  <xacro:cylinder_obj name_obj="obj5" dist_x="0.6" dist_z="0.45" color="green"/>
+  <xacro:cylinder_obj name_obj="obj6" dist_x="-0.6" dist_z="0.65" color="blue"/>
+  <xacro:cylinder_obj name_obj="obj7" dist_x="-0.3" dist_z="0.65" color="blue"/>
+  <xacro:cylinder_obj name_obj="obj8" dist_x="0.0" dist_z="0.65" color="blue"/>
+  <xacro:cylinder_obj name_obj="obj9" dist_x="0.3" dist_z="0.65" color="blue"/>
+  <xacro:cylinder_obj name_obj="obj10" dist_x="0.6" dist_z="0.65" color="blue"/>
+  <xacro:cylinder_obj name_obj="obj11" dist_x="-0.6" dist_z="0.85" color="red"/>
+  <xacro:cylinder_obj name_obj="obj12" dist_x="-0.3" dist_z="0.85" color="red"/>
+  <xacro:cylinder_obj name_obj="obj13" dist_x="0.0" dist_z="0.85" color="red"/>
+  <xacro:cylinder_obj name_obj="obj14" dist_x="0.3" dist_z="0.85" color="red"/>
+  <xacro:cylinder_obj name_obj="obj15" dist_x="0.6" dist_z="0.85" color="red"/>
   <xacro:include filename="$(find robot_description)/urdf/obj_gazebo.xacro"/>
 </robot>

File: robot_description/urdf/obj_gazebo.xacro (robot description, xacro)
@@ -31,17 +31,17 @@
   </gazebo>
   <gazebo reference="obj1">
-    <material>Gazebo/Blue</material>
+    <material>Gazebo/Green</material>
   </gazebo>
   <gazebo reference="obj2">
-    <material>Gazebo/Blue</material>
+    <material>Gazebo/Green</material>
   </gazebo>
   <gazebo reference="obj3">
-    <material>Gazebo/Blue</material>
+    <material>Gazebo/Green</material>
   </gazebo>
   <gazebo reference="obj4">
-    <material>Gazebo/Blue</material>
+    <material>Gazebo/Green</material>
   </gazebo>
   <gazebo reference="obj5">
-    <material>Gazebo/Blue</material>
+    <material>Gazebo/Green</material>
   </gazebo>
   <gazebo reference="obj6">
@@ -61,17 +61,17 @@
   </gazebo>
   <gazebo reference="obj11">
-    <material>Gazebo/Blue</material>
+    <material>Gazebo/Red</material>
   </gazebo>
   <gazebo reference="obj12">
-    <material>Gazebo/Blue</material>
+    <material>Gazebo/Red</material>
   </gazebo>
   <gazebo reference="obj13">
-    <material>Gazebo/Blue</material>
+    <material>Gazebo/Red</material>
   </gazebo>
   <gazebo reference="obj14">
-    <material>Gazebo/Blue</material>
+    <material>Gazebo/Red</material>
   </gazebo>
   <gazebo reference="obj15">
-    <material>Gazebo/Blue</material>
+    <material>Gazebo/Red</material>
   </gazebo>
 </robot>

File: robot_description/urdf/parameter.xacro (robot description, xacro)
@@ -44,5 +44,14 @@
   </material>
   <material name="blue">
-    <color rgba="${118/255} ${186/255} ${255/255} 0.62"/>
+    <color rgba="${146/255} ${195/255} ${255/255} 0.8"/>
+  </material>
+  <material name="red">
+    <color rgba="${255/255} ${51/255} ${51/255} 0.8"/>
+  </material>
+  <material name="yellow">
+    <color rgba="${215/255} ${196/255} ${23/255} 0.8"/>
+  </material>
+  <material name="green">
+    <color rgba="${0/255} ${168/255} ${44/255} 0.8"/>
   </material>
 </robot>
