Commit message: divide xacro file

File: robot_description/urdf/gazebo.xacro (robot description, xacro)
@@ -6,17 +6,63 @@
           filename="libgazebo_ros_joint_state_publisher.so">
           <update_rate>20</update_rate>
+          <joint_name>joint0</joint_name>
           <joint_name>joint1</joint_name>
           <joint_name>joint2</joint_name>
+          <joint_name>joint3</joint_name>
+          <joint_name>joint4</joint_name>
+          <joint_name>joint5</joint_name>
+          <joint_name>joint6</joint_name>
       </plugin>
   </gazebo>
   <ros2_control name="GazeboSystem" type="system">
     <hardware>
-        <!-- <plugin>ros2_control_demo_example_3/RRBotSystemMultiInterfaceHardware</plugin>
-        <param name="example_param_hw_start_duration_sec">0.0</param>
-        <param name="example_param_hw_stop_duration_sec">3.0</param>
-        <param name="example_param_hw_slowdown">${slowdown}</param> -->
       <plugin>gazebo_ros2_control/GazeboSystem</plugin>
     </hardware>
+    <joint name="joint0">
+        <command_interface name="position">
+          <param name="min">-0.75</param>
+          <param name="max">0.75</param>
+        </command_interface>
+        <state_interface name="position">
+            <param name="initial_value">0.0</param>
+        </state_interface>
+    </joint>
     <joint name="joint1">
+        <command_interface name="position">
+          <param name="min">-3.14</param>
+          <param name="max">3.14</param>
+        </command_interface>
+        <state_interface name="position">
+            <param name="initial_value">0.0</param>
+        </state_interface>
+    </joint>
+    <joint name="joint2">
+        <command_interface name="position">
+          <param name="min">-3.14</param>
+          <param name="max">3.14</param>
+        </command_interface>
+        <state_interface name="position">
+            <param name="initial_value">0.0</param>
+        </state_interface>
+    </joint>
+    <joint name="joint3">
+        <command_interface name="position">
+          <param name="min">-3.14</param>
+          <param name="max">3.14</param>
+        </command_interface>
+        <state_interface name="position">
+            <param name="initial_value">0.0</param>
+        </state_interface>
+    </joint>
+    <joint name="joint4">
+        <command_interface name="position">
+          <param name="min">-3.14</param>
+          <param name="max">3.14</param>
+        </command_interface>
+        <state_interface name="position">
+            <param name="initial_value">0.0</param>
+        </state_interface>
+    </joint>
+    <joint name="joint5">
         <command_interface name="position">
           <param name="min">-1</param>
@@ -26,37 +72,46 @@
             <param name="initial_value">0.0</param>
         </state_interface>
-        <state_interface name="velocity"/>
-        <state_interface name="effort"/>
     </joint>
-    <joint name="joint2">
+    <joint name="joint6">
         <command_interface name="position">
-          <param name="min">-1</param>
-          <param name="max">1</param>
+          <param name="min">-3.14</param>
+          <param name="max">3.14</param>
         </command_interface>
         <state_interface name="position">
             <param name="initial_value">0.0</param>
         </state_interface>
-        <state_interface name="velocity"/>
-        <state_interface name="effort"/>
     </joint>
   </ros2_control>
   <gazebo>
-    <plugin name="gazebo_ros_control" filename="libgazebo_ros_control.so">
+    <plugin name="gazebo_ros2_control" filename="libgazebo_ros2_control.so">
       <parameters>$(find robot_description)/config/controller.yaml</parameters>
-      <robotNamespace>/robot</robotNamespace>
     </plugin>
   </gazebo>
   <!-- Base Link -->
-  <gazebo reference="base_link">
+  <gazebo reference="shelf">
     <material>Gazebo/White</material>
   </gazebo>
-  <!-- Link1 -->
+  <gazebo reference="obj1">
+    <material>Gazebo/Blue</material>
+  </gazebo>
+  <gazebo reference="obj2 ">
+    <material>Gazebo/Blue</material>
+  </gazebo>
+  <gazebo reference="obj8">
+    <material>Gazebo/Blue</material>
+  </gazebo>
+  <gazebo reference="link_slide">
+    <material>Gazebo/White</material>
+  </gazebo>
+  <gazebo reference="link0">
+    <material>Gazebo/White</material>
+  </gazebo>
   <gazebo reference="link1">
     <material>Gazebo/White</material>
   </gazebo>
-  <gazebo reference="joint_link1">
+  <gazebo reference="link_joint2-1">
     <material>Gazebo/Orange</material>
   </gazebo>
-  <gazebo reference="joint_link2">
+  <gazebo reference="link_joint2-2">
     <material>Gazebo/Orange</material>
   </gazebo>
@@ -64,3 +119,27 @@
     <material>Gazebo/White</material>
   </gazebo>
+  <gazebo reference="link_joint3-1">
+    <material>Gazebo/Orange</material>
+  </gazebo>
+  <gazebo reference="link_joint3-2">
+    <material>Gazebo/Orange</material>
+  </gazebo>
+  <gazebo reference="link3">
+    <material>Gazebo/White</material>
+  </gazebo>
+  <gazebo reference="link_joint4">
+    <material>Gazebo/Orange</material>
+  </gazebo>
+  <gazebo reference="link4">
+    <material>Gazebo/White</material>
+  </gazebo>
+  <gazebo reference="link_joint5">
+    <material>Gazebo/Orange</material>
+  </gazebo>
+  <gazebo reference="link5">
+    <material>Gazebo/White</material>
+  </gazebo>
+  <gazebo reference="link_hook">
+    <material>Gazebo/Orange</material>
+  </gazebo>
 </robot>

File: robot_description/urdf/robot.xacro (robot description, xacro)
@@ -1,178 +1,9 @@
 <?xml version="1.0"?>
 <robot name="robot" xmlns:xacro="http://www.ros.org/wiki/xacro">
-  <xacro:property name="PI" value="3.1415926535897931"/>
-  <xacro:property name="shelf_dist" value="0.1"/>
-  <xacro:property name="params_path" value="$(find robot_description)/config/properties.yaml"/>
-  <xacro:property name="params" value="${xacro.load_yaml(params_path)}"/>
-  <xacro:property name="LINK1" value="${params['link1_length']}"/>
-  <xacro:property name="LINK2" value="${params['link2_length']}"/>
-  <xacro:property name="LINK3" value="${params['link3_length']}"/>
-  <xacro:property name="LINK4" value="${params['link4_length']}"/>
-  <xacro:property name="LINK5" value="${params['link5_length']}"/>
-  <xacro:property name="MAX_LINK1" value="0.2"/>
-  <xacro:property name="MAX_LINK2" value="0.2"/>
-  <xacro:property name="MAX_LINK3" value="0.2"/>
-  <xacro:property name="MAX_LINK4" value="0.2"/>
-  <xacro:property name="MAX_LINK5" value="0.2"/>
-  <xacro:property name="MIN_LINK1" value="0.045"/>
-  <xacro:property name="MIN_LINK2" value="0.085"/>
-  <xacro:property name="MIN_LINK3" value="0.05125"/>
-  <xacro:property name="MIN_LINK4" value="0.045"/>
-  <xacro:property name="MIN_LINK5" value="0.0115"/>
-  <xacro:if value="${LINK1 >= MAX_LINK1}">
-    <xacro:property name="LINK1" value="${MAX_LINK1}"/>
-  </xacro:if>
-  <xacro:if value="${MIN_LINK1 >= LINK1}">
-    <xacro:property name="LINK1" value="${MIN_LINK1}"/>
-  </xacro:if>
-  <xacro:if value="${LINK2 >= MAX_LINK2}">
-    <xacro:property name="LINK2" value="${MAX_LINK2}"/>
-  </xacro:if>
-  <xacro:if value="${MIN_LINK2 >= LINK2}">
-    <xacro:property name="LINK2" value="${MIN_LINK2}"/>
-  </xacro:if>
-  <xacro:if value="${LINK3 >= MAX_LINK3}">
-    <xacro:property name="LINK3" value="${MAX_LINK3}"/>
-  </xacro:if>
-  <xacro:if value="${MIN_LINK3 >= LINK3}">
-    <xacro:property name="LINK3" value="${MIN_LINK3}"/>
-  </xacro:if>
-  <xacro:if value="${LINK4 >= MAX_LINK4}">
-    <xacro:property name="LINK4" value="${MAX_LINK4}"/>
-  </xacro:if>
-  <xacro:if value="${MIN_LINK1 >= LINK4}">
-    <xacro:property name="LINK4" value="${MIN_LINK4}"/>
-  </xacro:if>
-  <xacro:if value="${LINK5 >= MAX_LINK5}">
-    <xacro:property name="LINK5" value="${MAX_LINK5}"/>
-  </xacro:if>
-  <xacro:if value="${MIN_LINK5 >= LINK5}">
-    <xacro:property name="LINK5" value="${MIN_LINK5}"/>
-  </xacro:if>
-  <xacro:property name="LINK1_LENGTH" value="${LINK1-0.045}"/>
-  <xacro:property name="LINK2_LENGTH" value="${LINK2-0.085}"/>
-  <xacro:property name="LINK3_LENGTH" value="${LINK3-0.045-0.00625}"/>
-  <xacro:property name="LINK4_LENGTH" value="${LINK4-0.045}"/>
-  <xacro:property name="LINK5_LENGTH" value="${LINK5+0.015}"/>
-  <material name="orange">
-    <color rgba="${255/255} ${108/255} ${10/255} 1.0"/>
-  </material>
-  <material name="white">
-    <color rgba="1.0 1.0 1.0 1.0"/>
-  </material>
-  <material name="blue">
-    <color rgba="${118/255} ${186/255} ${255/255} 0.62"/>
-  </material>
+  <!-- parameter -->
+  <xacro:include filename="$(find robot_description)/urdf/parameter.xacro"/>
   <link name="world"/>
-  <joint name="fixed_shelf" type="fixed">
-    <parent link="world"/>
-    <child link="shelf"/>
-  </joint>
-  <link name="shelf">
-    <visual>
-      <origin xyz="0 ${shelf_dist+0.1} 0" rpy="0 0 0"/>
-      <geometry>
-        <mesh filename="file:///$(find robot_description)/meshes/shelf.STL"/>
-      </geometry>
-      <material name="white"/>
-    </visual>
-    <inertial>
-      <origin xyz="0 ${shelf_dist+0.1} 0" rpy="0 0 0"/>
-      <mass value="5.0"/>
-      <inertia
-        ixx="0.01" ixy="0.0" ixz="0.0"
-        iyy="0.01" iyz="0.0"
-        izz="0.01"/>
-    </inertial>
-    <collision>
-      <origin xyz="0 ${shelf_dist+0.1} 0" rpy="0 0 0"/>
-      <geometry>
-        <mesh filename="file:///$(find robot_description)/meshes/shelf.STL"/>
-      </geometry>
-    </collision>
-  </link>
-  <joint name="float_obj1" type="floating">
-    <parent link="shelf"/>
-    <child link="obj1"/>
-    <dynamics damping="0.0" friction="10.0"/>
-    <limit effort="1" velocity="1.0" lower="-2.2" upper="0.7" />
-  </joint>
-  <link name="obj1">
-    <visual>
-      <origin xyz="-0.6 ${shelf_dist+0.35} 0.45" rpy="0 0 0"/>
-      <geometry>
-        <cylinder radius="0.04" length="0.1"/>
-      </geometry>
-      <material name="blue"/>
-    </visual>
-    <inertial>
-      <origin xyz="-0.6 ${shelf_dist+0.35} 0.45" rpy="0 0 0"/>
-      <mass value="0.01"/>
-      <inertia
-        ixx="0.01" ixy="0.0" ixz="0.0"
-        iyy="0.01" iyz="0.0"
-        izz="0.01"/>
-    </inertial>
-    <collision>
-      <origin xyz="-0.6 ${shelf_dist+0.35} 0.45" rpy="0 0 0"/>
-      <geometry>
-        <cylinder radius="0.04" length="0.1"/>
-      </geometry>
-    </collision>
-  </link>
-  <joint name="float_obj2" type="floating">
-    <parent link="shelf"/>
-    <child link="obj2"/>
-  </joint>
-  <link name="obj2">
-    <visual>
-      <origin xyz="-0.3 ${shelf_dist+0.35} 0.45" rpy="0 0 0"/>
-      <geometry>
-        <cylinder radius="0.04" length="0.1"/>
-      </geometry>
-      <material name="blue"/>
-    </visual>
-    <inertial>
-      <origin xyz="-0.3 ${shelf_dist+0.35} 0.45" rpy="0 0 0"/>
-      <mass value="0.01"/>
-      <inertia
-        ixx="0.01" ixy="0.0" ixz="0.0"
-        iyy="0.01" iyz="0.0"
-        izz="0.01"/>
-    </inertial>
-    <collision>
-      <origin xyz="-0.3 ${shelf_dist+0.35} 0.45" rpy="0 0 0"/>
-      <geometry>
-        <cylinder radius="0.04" length="0.1"/>
-      </geometry>
-    </collision>
-  </link>
-  <joint name="float_obj8" type="fixed">
-    <parent link="shelf"/>
-    <child link="obj8"/>
-  </joint>
-  <link name="obj8">
-    <visual>
-      <origin xyz="0.0 ${shelf_dist+0.35} 0.85" rpy="0 0 0"/>
-      <geometry>
-        <cylinder radius="0.04" length="0.1"/>
-      </geometry>
-      <material name="blue"/>
-    </visual>
-    <inertial>
-      <origin xyz="0.0 ${shelf_dist+0.35} 0.85" rpy="0 0 0"/>
-      <mass value="0.01"/>
-      <inertia
-        ixx="0.01" ixy="0.0" ixz="0.0"
-        iyy="0.01" iyz="0.0"
-        izz="0.01"/>
-    </inertial>
-    <collision>
-      <origin xyz="0.0 ${shelf_dist+0.35} 0.85" rpy="0 0 0"/>
-      <geometry>
-        <cylinder radius="0.04" length="0.1"/>
-      </geometry>
-    </collision>
-  </link>
+  <!-- world -->
+  <xacro:include filename="$(find robot_description)/urdf/world.xacro"/>
   <!-- robot -->
   <joint name="fixed_robot" type="fixed">
@@ -227,10 +58,4 @@
         izz="0.01"/>
     </inertial>
-    <!-- <collision>
-      <origin xyz="0.0 0.0 0.0" rpy="0.0 0.0 0.0"/>
-      <geometry>
-        <mesh filename="file:///$(find robot_description)/meshes/link_base.STL"/>
-      </geometry>
-    </collision> -->
   </link>
   <joint name="joint1" type="revolute">
@@ -578,146 +403,5 @@
     </collision>
   </link>
-  <!-- <xacro:include filename="gazebo.xacro" /> -->
   <!-- gazebo plugin -->
-  <gazebo>
-      <plugin name="gazebo_ros_joint_state_publisher"
-          filename="libgazebo_ros_joint_state_publisher.so">
-          <update_rate>20</update_rate>
-          <joint_name>joint0</joint_name>
-          <joint_name>joint1</joint_name>
-          <joint_name>joint2</joint_name>
-          <joint_name>joint3</joint_name>
-          <joint_name>joint4</joint_name>
-          <joint_name>joint5</joint_name>
-          <joint_name>joint6</joint_name>
-      </plugin>
-  </gazebo>
-  <ros2_control name="GazeboSystem" type="system">
-    <hardware>
-      <plugin>gazebo_ros2_control/GazeboSystem</plugin>
-    </hardware>
-    <joint name="joint0">
-        <command_interface name="position">
-          <param name="min">-0.75</param>
-          <param name="max">0.75</param>
-        </command_interface>
-        <state_interface name="position">
-            <param name="initial_value">0.0</param>
-        </state_interface>
-    </joint>
-    <joint name="joint1">
-        <command_interface name="position">
-          <param name="min">-3.14</param>
-          <param name="max">3.14</param>
-        </command_interface>
-        <state_interface name="position">
-            <param name="initial_value">0.0</param>
-        </state_interface>
-    </joint>
-    <joint name="joint2">
-        <command_interface name="position">
-          <param name="min">-3.14</param>
-          <param name="max">3.14</param>
-        </command_interface>
-        <state_interface name="position">
-            <param name="initial_value">0.0</param>
-        </state_interface>
-    </joint>
-    <joint name="joint3">
-        <command_interface name="position">
-          <param name="min">-3.14</param>
-          <param name="max">3.14</param>
-        </command_interface>
-        <state_interface name="position">
-            <param name="initial_value">0.0</param>
-        </state_interface>
-    </joint>
-    <joint name="joint4">
-        <command_interface name="position">
-          <param name="min">-3.14</param>
-          <param name="max">3.14</param>
-        </command_interface>
-        <state_interface name="position">
-            <param name="initial_value">0.0</param>
-        </state_interface>
-    </joint>
-    <joint name="joint5">
-        <command_interface name="position">
-          <param name="min">-1</param>
-          <param name="max">1</param>
-        </command_interface>
-        <state_interface name="position">
-            <param name="initial_value">0.0</param>
-        </state_interface>
-    </joint>
-    <joint name="joint6">
-        <command_interface name="position">
-          <param name="min">-3.14</param>
-          <param name="max">3.14</param>
-        </command_interface>
-        <state_interface name="position">
-            <param name="initial_value">0.0</param>
-        </state_interface>
-    </joint>
-  </ros2_control>
-  <gazebo>
-    <plugin name="gazebo_ros2_control" filename="libgazebo_ros2_control.so">
-      <parameters>$(find robot_description)/config/controller.yaml</parameters>
-    </plugin>
-  </gazebo>
-  <!-- Base Link -->
-  <gazebo reference="shelf">
-    <material>Gazebo/White</material>
-  </gazebo>
-  <gazebo reference="obj1">
-    <material>Gazebo/Blue</material>
-  </gazebo>
-  <gazebo reference="obj2 ">
-    <material>Gazebo/Blue</material>
-  </gazebo>
-  <gazebo reference="obj8">
-    <material>Gazebo/Blue</material>
-  </gazebo>
-  <gazebo reference="link_slide">
-    <material>Gazebo/White</material>
-  </gazebo>
-  <gazebo reference="link0">
-    <material>Gazebo/White</material>
-  </gazebo>
-  <gazebo reference="link1">
-    <material>Gazebo/White</material>
-  </gazebo>
-  <gazebo reference="link_joint2-1">
-    <material>Gazebo/Orange</material>
-  </gazebo>
-  <gazebo reference="link_joint2-2">
-    <material>Gazebo/Orange</material>
-  </gazebo>
-  <gazebo reference="link2">
-    <material>Gazebo/White</material>
-  </gazebo>
-  <gazebo reference="link_joint3-1">
-    <material>Gazebo/Orange</material>
-  </gazebo>
-  <gazebo reference="link_joint3-2">
-    <material>Gazebo/Orange</material>
-  </gazebo>
-  <gazebo reference="link3">
-    <material>Gazebo/White</material>
-  </gazebo>
-  <gazebo reference="link_joint4">
-    <material>Gazebo/Orange</material>
-  </gazebo>
-  <gazebo reference="link4">
-    <material>Gazebo/White</material>
-  </gazebo>
-  <gazebo reference="link_joint5">
-    <material>Gazebo/Orange</material>
-  </gazebo>
-  <gazebo reference="link5">
-    <material>Gazebo/White</material>
-  </gazebo>
-  <gazebo reference="link_hook">
-    <material>Gazebo/Orange</material>
-  </gazebo>
+  <xacro:include filename="$(find robot_description)/urdf/gazebo.xacro"/>
 </robot>
