Commit message: test script shell

File: robot_description/urdf/gazebo.xacro (robot description, xacro)
@@ -6,9 +6,8 @@
           filename="libgazebo_ros_joint_state_publisher.so">
           <update_rate>20</update_rate>
-          <joint_name>joint0</joint_name>
+          <joint_name>jointX</joint_name>
+          <joint_name>jointY</joint_name>
+          <joint_name>jointZ</joint_name>
           <joint_name>joint1</joint_name>
-          <joint_name>joint2</joint_name>
-          <joint_name>joint3</joint_name>
-          <joint_name>joint4</joint_name>
           <joint_name>joint5</joint_name>
           <joint_name>joint6</joint_name>
@@ -19,11 +18,29 @@
       <plugin>gazebo_ros2_control/GazeboSystem</plugin>
     </hardware>
-    <joint name="joint0">
+    <joint name="jointX">
+        <command_interface name="position">
+          <param name="min">-0.95</param>
+          <param name="max">0.95</param>
+        </command_interface>
+        <command_interface name="velocity"/>
+        <state_interface name="position">
+        </state_interface>
+    </joint>
+    <joint name="jointY">
         <command_interface name="position">
           <param name="min">-0.75</param>
           <param name="max">0.75</param>
         </command_interface>
+        <command_interface name="velocity"/>
         <state_interface name="position">
-            <param name="initial_value">0.0</param>
+        </state_interface>
+    </joint>
+    <joint name="jointZ">
+        <command_interface name="position">
+          <param name="min">0</param>
+          <param name="max">0.6</param>
+        </command_interface>
+        <command_interface name="velocity"/>
+        <state_interface name="position">
         </state_interface>
     </joint>
@@ -33,33 +50,6 @@
           <param name="max">3.14</param>
         </command_interface>
+        <command_interface name="velocity"/>
         <state_interface name="position">
-            <param name="initial_value">0.0</param>
-        </state_interface>
-    </joint>
-    <joint name="joint2">
-        <command_interface name="position">
-          <param name="min">-3.14</param>
-          <param name="max">3.14</param>
-        </command_interface>
-        <state_interface name="position">
-            <param name="initial_value">0.0</param>
-        </state_interface>
-    </joint>
-    <joint name="joint3">
-        <command_interface name="position">
-          <param name="min">-3.14</param>
-          <param name="max">3.14</param>
-        </command_interface>
-        <state_interface name="position">
-            <param name="initial_value">0.0</param>
-        </state_interface>
-    </joint>
-    <joint name="joint4">
-        <command_interface name="position">
-          <param name="min">-3.14</param>
-          <param name="max">3.14</param>
-        </command_interface>
-        <state_interface name="position">
-            <param name="initial_value">0.0</param>
         </state_interface>
     </joint>
@@ -69,6 +59,6 @@
           <param name="max">1</param>
         </command_interface>
+        <command_interface name="velocity"/>
         <state_interface name="position">
-            <param name="initial_value">0.0</param>
         </state_interface>
     </joint>
@@ -78,6 +68,6 @@
           <param name="max">3.14</param>
         </command_interface>
+        <command_interface name="velocity"/>
         <state_interface name="position">
-            <param name="initial_value">0.0</param>
         </state_interface>
     </joint>
@@ -85,20 +75,11 @@
   <gazebo>
     <plugin name="gazebo_ros2_control" filename="libgazebo_ros2_control.so">
-      <parameters>$(find robot_description)/config/controller_v1.yaml</parameters>
+      <parameters>$(find robot_description)/config/controller.yaml</parameters>
     </plugin>
   </gazebo>
   <!-- Base Link -->
-  <gazebo reference="shelf">
+  <!-- <gazebo reference="shelf">
     <material>Gazebo/White</material>
-  </gazebo>
-  <gazebo reference="obj1">
-    <material>Gazebo/Blue</material>
-  </gazebo>
-  <gazebo reference="obj2 ">
-    <material>Gazebo/Blue</material>
-  </gazebo>
-  <gazebo reference="obj8">
-    <material>Gazebo/Blue</material>
-  </gazebo>
+  </gazebo> -->
   <gazebo reference="link0">
     <material>Gazebo/White</material>
@@ -116,18 +97,6 @@
     <material>Gazebo/White</material>
   </gazebo>
-  <gazebo reference="link_joint3-1">
-    <material>Gazebo/Orange</material>
-  </gazebo>
-  <gazebo reference="link_joint3-2">
-    <material>Gazebo/Orange</material>
-  </gazebo>
-  <gazebo reference="link3">
-    <material>Gazebo/White</material>
-  </gazebo>
   <gazebo reference="link_joint4">
     <material>Gazebo/Orange</material>
-  </gazebo>
-  <gazebo reference="link4">
-    <material>Gazebo/White</material>
   </gazebo>
   <gazebo reference="link_joint5">
@@ -137,5 +106,5 @@
     <material>Gazebo/White</material>
   </gazebo>
-  <gazebo reference="link_hook">
+  <gazebo reference="end_effector">
     <material>Gazebo/Orange</material>
   </gazebo>

File: robot_description/urdf/parameter.xacro (robot description, xacro)
@@ -3,5 +3,5 @@
   <xacro:property name="shelf_dist" value="0.2"/>
   <xacro:property name="cylinder_obj_mass" value="0.01"/>
-  <xacro:property name="params_path" value="$(find robot_description)/config/properties_v2.yaml"/>
+  <xacro:property name="params_path" value="$(find robot_description)/config/properties.yaml"/>
   <xacro:property name="params" value="${xacro.load_yaml(params_path)}"/>
   <xacro:property name="LINK1" value="${params['link1_length']}"/>

File: robot_description/urdf/robot.xacro (robot description, xacro)
@@ -2,5 +2,5 @@
 <robot name="robot" xmlns:xacro="http://www.ros.org/wiki/xacro">
   <!-- parameter -->
-  <xacro:include filename="$(find robot_description)/urdf/parameter_v2.xacro"/>
+  <xacro:include filename="$(find robot_description)/urdf/parameter.xacro"/>
   <link name="world"/>
   <!-- world -->
@@ -282,5 +282,5 @@
       <origin xyz="0 0 0" rpy="0 0 0"/>
       <geometry>
-        <mesh filename="file:///$(find robot_description)/meshes/end_effectorI.STL"/>
+        <mesh filename="file:///$(find robot_description)/meshes/end_effectorL.STL"/>
       </geometry>
       <material name="orange"/>
@@ -297,9 +297,9 @@
       <origin xyz="0.0 0.0 0.0" rpy="0.0 0.0 0.0"/>
       <geometry>
-        <mesh filename="file:///$(find robot_description)/meshes/end_effectorI.STL"/>
+        <mesh filename="file:///$(find robot_description)/meshes/end_effectorL.STL"/>
       </geometry>
     </collision>
   </link>
   <!-- gazebo plugin -->
-  <xacro:include filename="$(find robot_description)/urdf/gazebo_v2.xacro"/>
+  <xacro:include filename="$(find robot_description)/urdf/gazebo.xacro"/>
 </robot>

File: robot_description/urdf/spawn_obj.xacro (robot description, xacro)
@@ -1,5 +1,5 @@
 <?xml version="1.0"?>
 <robot name="cylinder_object" xmlns:xacro="http://www.ros.org/wiki/xacro">
-  <xacro:include filename="$(find robot_description)/urdf/parameter_v2.xacro"/>
+  <xacro:include filename="$(find robot_description)/urdf/parameter.xacro"/>
   <link name="world"/>
   <joint name="float_obj1" type="floating">

File: robot_description/urdf/world.xacro (robot description, xacro)
@@ -1,5 +1,5 @@
 <?xml version="1.0"?>
 <robot name="environment" xmlns:xacro="http://www.ros.org/wiki/xacro">
-  <xacro:include filename="$(find robot_description)/urdf/parameter_v2.xacro"/>
+  <xacro:include filename="$(find robot_description)/urdf/parameter.xacro"/>
   <link name="world"/>
   <joint name="fixed_shelf" type="fixed">

Commit message: Update 24.07.23

File: robot_description/urdf/gazebo.xacro (robot description, xacro)
@@ -79,7 +79,4 @@
   </gazebo>
   <!-- Base Link -->
-  <!-- <gazebo reference="shelf">
-    <material>Gazebo/White</material>
-  </gazebo> -->
   <gazebo reference="link0">
     <material>Gazebo/White</material>
