Commit message: update 25.07.23

File: robot_description/urdf/parameter.xacro (robot description, xacro)
@@ -55,3 +55,6 @@
     <color rgba="${0/255} ${168/255} ${44/255} 0.8"/>
   </material>
+  <material name="black">
+    <color rgba="${0/255} ${0/255} ${0/255} 0.8"/>
+  </material>
 </robot>

File: robot_description/urdf/world.xacro (robot description, xacro)
@@ -17,9 +17,9 @@
     <inertial>
       <origin xyz="0 ${shelf_dist+0.1} 0" rpy="0 0 0"/>
-      <mass value="1000.0"/>
+      <mass value="316"/>
       <inertia
-        ixx="0.01" ixy="0.0" ixz="0.0"
-        iyy="0.01" iyz="0.0"
-        izz="0.01"/>
+        ixx="68.8" ixy="7.56" ixz="-0.58"
+        iyy="148.1" iyz="-6.9"
+        izz="182.29"/>
     </inertial>
     <collision>
