Commit message: update game logic

File: robot_description/urdf/charcoal.xacro (robot description, xacro)
@@ -1,4 +1,4 @@
 <?xml version="1.0"?>
-<robot name="cylinder_object" xmlns:xacro="http://www.ros.org/wiki/xacro">
+<robot name="charcoal" xmlns:xacro="http://www.ros.org/wiki/xacro">
   <xacro:include filename="$(find robot_description)/urdf/parameter.xacro"/>
   <xacro:property name="IXX" value="${((cylinder_obj_mass*0.04*0.04)/4)+((cylinder_obj_mass*0.1*0.1)/12)}"/>
@@ -6,7 +6,7 @@
   <xacro:property name="IZZ" value="${(cylinder_obj_mass*0.04*0.04)/2}"/>
   <link name="world"/>
-  <xacro:macro name="cylinder_obj" params="name_obj dist_x dist_z color">
+  <xacro:macro name="cylinder_obj" params="name_obj dist_x dist_y dist_z color">
     <joint name="${name_obj}_prisX" type="prismatic">
-        <origin xyz="${dist_x} ${shelf_dist+0.35} ${dist_z}" rpy="0.0 0.0 0.0"/>
+        <origin xyz="${dist_x} ${shelf_dist+dist_y} ${dist_z}" rpy="0.0 0.0 0.0"/>
         <parent link="world"/>
         <child link="${name_obj}_slideX"/>
@@ -129,19 +129,6 @@
     </link>
   </xacro:macro>
-  <xacro:cylinder_obj name_obj="obj1" dist_x="-0.6" dist_z="0.45" color="green"/>
-  <xacro:cylinder_obj name_obj="obj2" dist_x="-0.3" dist_z="0.45" color="green"/>
-  <xacro:cylinder_obj name_obj="obj3" dist_x="0.0" dist_z="0.45" color="green"/>
-  <xacro:cylinder_obj name_obj="obj4" dist_x="0.3" dist_z="0.45" color="green"/>
-  <xacro:cylinder_obj name_obj="obj5" dist_x="0.6" dist_z="0.45" color="green"/>
-  <xacro:cylinder_obj name_obj="obj6" dist_x="-0.6" dist_z="0.65" color="blue"/>
-  <xacro:cylinder_obj name_obj="obj7" dist_x="-0.3" dist_z="0.65" color="blue"/>
-  <xacro:cylinder_obj name_obj="obj8" dist_x="0.0" dist_z="0.65" color="blue"/>
-  <xacro:cylinder_obj name_obj="obj9" dist_x="0.3" dist_z="0.65" color="blue"/>
-  <xacro:cylinder_obj name_obj="obj10" dist_x="0.6" dist_z="0.65" color="blue"/>
-  <xacro:cylinder_obj name_obj="obj11" dist_x="-0.6" dist_z="0.85" color="red"/>
-  <xacro:cylinder_obj name_obj="obj12" dist_x="-0.3" dist_z="0.85" color="red"/>
-  <xacro:cylinder_obj name_obj="obj13" dist_x="0.0" dist_z="0.85" color="red"/>
-  <xacro:cylinder_obj name_obj="obj14" dist_x="0.3" dist_z="0.85" color="red"/>
-  <xacro:cylinder_obj name_obj="obj15" dist_x="0.6" dist_z="0.85" color="red"/>
-  <xacro:include filename="$(find robot_description)/urdf/obj_gazebo.xacro"/>
+  <xacro:cylinder_obj name_obj="objR" dist_x="-0.85" dist_y="0.0" dist_z="0.45" color="black"/>
+  <xacro:cylinder_obj name_obj="objL" dist_x="0.85" dist_y="0.0" dist_z="0.45" color="black"/>
+  <xacro:include filename="$(find robot_description)/urdf/charcoal_gazebo.xacro"/>
 </robot>

File: robot_description/urdf/cylinder_gazebo.xacro (robot description, xacro)
@@ -13,7 +13,67 @@
       <plugin name="gazebo_ros_joint_state_publisher_cylinder"
           filename="libgazebo_ros_joint_state_publisher.so">
+          <xacro:cylider_gazebo name_obj="obj1"/>
+          <xacro:cylider_gazebo name_obj="obj2"/>
+          <xacro:cylider_gazebo name_obj="obj3"/>
+          <xacro:cylider_gazebo name_obj="obj4"/>
+          <xacro:cylider_gazebo name_obj="obj5"/>
+          <xacro:cylider_gazebo name_obj="obj6"/>
+          <xacro:cylider_gazebo name_obj="obj7"/>
+          <xacro:cylider_gazebo name_obj="obj8"/>
+          <xacro:cylider_gazebo name_obj="obj9"/>
+          <xacro:cylider_gazebo name_obj="obj10"/>
+          <xacro:cylider_gazebo name_obj="obj11"/>
+          <xacro:cylider_gazebo name_obj="obj12"/>
+          <xacro:cylider_gazebo name_obj="obj13"/>
+          <xacro:cylider_gazebo name_obj="obj14"/>
+          <xacro:cylider_gazebo name_obj="obj15"/>
           <xacro:cylider_gazebo name_obj="objR"/>
           <xacro:cylider_gazebo name_obj="objL"/>
       </plugin>
+  </gazebo>
+  <gazebo reference="obj1">
+    <material>Gazebo/Green</material>
+  </gazebo>
+  <gazebo reference="obj2">
+    <material>Gazebo/Green</material>
+  </gazebo>
+  <gazebo reference="obj3">
+    <material>Gazebo/Green</material>
+  </gazebo>
+  <gazebo reference="obj4">
+    <material>Gazebo/Green</material>
+  </gazebo>
+  <gazebo reference="obj5">
+    <material>Gazebo/Green</material>
+  </gazebo>
+  <gazebo reference="obj6">
+    <material>Gazebo/Blue</material>
+  </gazebo>
+  <gazebo reference="obj7">
+    <material>Gazebo/Blue</material>
+  </gazebo>
+  <gazebo reference="obj8">
+    <material>Gazebo/Blue</material>
+  </gazebo>
+  <gazebo reference="obj9">
+    <material>Gazebo/Blue</material>
+  </gazebo>
+  <gazebo reference="obj10">
+    <material>Gazebo/Blue</material>
+  </gazebo>
+  <gazebo reference="obj11">
+    <material>Gazebo/Red</material>
+  </gazebo>
+  <gazebo reference="obj12">
+    <material>Gazebo/Red</material>
+  </gazebo>
+  <gazebo reference="obj13">
+    <material>Gazebo/Red</material>
+  </gazebo>
+  <gazebo reference="obj14">
+    <material>Gazebo/Red</material>
+  </gazebo>
+  <gazebo reference="obj15">
+    <material>Gazebo/Red</material>
   </gazebo>
   <gazebo reference="objR">

File: robot_description/urdf/obj.xacro (robot description, xacro)
@@ -1,4 +1,4 @@
 <?xml version="1.0"?>
-<robot name="cylinder" xmlns:xacro="http://www.ros.org/wiki/xacro">
+<robot name="obj" xmlns:xacro="http://www.ros.org/wiki/xacro">
   <xacro:include filename="$(find robot_description)/urdf/parameter.xacro"/>
   <xacro:property name="IXX" value="${((cylinder_obj_mass*0.04*0.04)/4)+((cylinder_obj_mass*0.1*0.1)/12)}"/>
@@ -6,7 +6,7 @@
   <xacro:property name="IZZ" value="${(cylinder_obj_mass*0.04*0.04)/2}"/>
   <link name="world"/>
-  <xacro:macro name="cylinder_obj" params="name_obj dist_x dist_y dist_z color">
+  <xacro:macro name="cylinder_obj" params="name_obj dist_x dist_z color">
     <joint name="${name_obj}_prisX" type="prismatic">
-        <origin xyz="${dist_x} ${shelf_dist+dist_y} ${dist_z}" rpy="0.0 0.0 0.0"/>
+        <origin xyz="${dist_x} ${shelf_dist+0.35} ${dist_z}" rpy="0.0 0.0 0.0"/>
         <parent link="world"/>
         <child link="${name_obj}_slideX"/>
@@ -129,21 +129,19 @@
     </link>
   </xacro:macro>
-  <xacro:cylinder_obj name_obj="obj1" dist_x="-0.6" dist_y="0.35" dist_z="0.45" color="green"/>
-  <xacro:cylinder_obj name_obj="obj2" dist_x="-0.3" dist_y="0.35" dist_z="0.45" color="green"/>
-  <xacro:cylinder_obj name_obj="obj3" dist_x="0.0" dist_y="0.35" dist_z="0.45" color="green"/>
-  <xacro:cylinder_obj name_obj="obj4" dist_x="0.3" dist_y="0.35" dist_z="0.45" color="green"/>
-  <xacro:cylinder_obj name_obj="obj5" dist_x="0.6" dist_y="0.35" dist_z="0.45" color="green"/>
-  <xacro:cylinder_obj name_obj="obj6" dist_x="-0.6" dist_y="0.35" dist_z="0.65" color="blue"/>
-  <xacro:cylinder_obj name_obj="obj7" dist_x="-0.3" dist_y="0.35" dist_z="0.65" color="blue"/>
-  <xacro:cylinder_obj name_obj="obj8" dist_x="0.0" dist_y="0.35" dist_z="0.65" color="blue"/>
-  <xacro:cylinder_obj name_obj="obj9" dist_x="0.3" dist_y="0.35" dist_z="0.65" color="blue"/>
-  <xacro:cylinder_obj name_obj="obj10" dist_x="0.6" dist_y="0.35" dist_z="0.65" color="blue"/>
-  <xacro:cylinder_obj name_obj="obj11" dist_x="-0.6" dist_y="0.35" dist_z="0.85" color="red"/>
-  <xacro:cylinder_obj name_obj="obj12" dist_x="-0.3" dist_y="0.35" dist_z="0.85" color="red"/>
-  <xacro:cylinder_obj name_obj="obj13" dist_x="0.0" dist_y="0.35" dist_z="0.85" color="red"/>
-  <xacro:cylinder_obj name_obj="obj14" dist_x="0.3" dist_y="0.35" dist_z="0.85" color="red"/>
-  <xacro:cylinder_obj name_obj="obj15" dist_x="0.6" dist_y="0.35" dist_z="0.85" color="red"/>
-  <xacro:cylinder_obj name_obj="objR" dist_x="-0.85" dist_y="0.0" dist_z="0.45" color="black"/>
-  <xacro:cylinder_obj name_obj="objL" dist_x="0.85" dist_y="0.0" dist_z="0.45" color="black"/>
-  <xacro:include filename="$(find robot_description)/urdf/cylinder_gazebo.xacro"/>
+  <xacro:cylinder_obj name_obj="obj1" dist_x="-0.6" dist_z="0.45" color="green"/>
+  <xacro:cylinder_obj name_obj="obj2" dist_x="-0.3" dist_z="0.45" color="green"/>
+  <xacro:cylinder_obj name_obj="obj3" dist_x="0.0" dist_z="0.45" color="green"/>
+  <xacro:cylinder_obj name_obj="obj4" dist_x="0.3" dist_z="0.45" color="green"/>
+  <xacro:cylinder_obj name_obj="obj5" dist_x="0.6" dist_z="0.45" color="green"/>
+  <xacro:cylinder_obj name_obj="obj6" dist_x="-0.6" dist_z="0.65" color="blue"/>
+  <xacro:cylinder_obj name_obj="obj7" dist_x="-0.3" dist_z="0.65" color="blue"/>
+  <xacro:cylinder_obj name_obj="obj8" dist_x="0.0" dist_z="0.65" color="blue"/>
+  <xacro:cylinder_obj name_obj="obj9" dist_x="0.3" dist_z="0.65" color="blue"/>
+  <xacro:cylinder_obj name_obj="obj10" dist_x="0.6" dist_z="0.65" color="blue"/>
+  <xacro:cylinder_obj name_obj="obj11" dist_x="-0.6" dist_z="0.85" color="red"/>
+  <xacro:cylinder_obj name_obj="obj12" dist_x="-0.3" dist_z="0.85" color="red"/>
+  <xacro:cylinder_obj name_obj="obj13" dist_x="0.0" dist_z="0.85" color="red"/>
+  <xacro:cylinder_obj name_obj="obj14" dist_x="0.3" dist_z="0.85" color="red"/>
+  <xacro:cylinder_obj name_obj="obj15" dist_x="0.6" dist_z="0.85" color="red"/>
+  <xacro:include filename="$(find robot_description)/urdf/obj_gazebo.xacro"/>
 </robot>
